File: KiCad Schematics and pcb/ESPHome AIO.kicad_sch (KiCad schematic)
At the start: 8 parts, among them IC1 ESP32-S3-WROOM-1-N8, J1 Conn_01x05, J2 Conn_02x12_Top_Bottom, J3 Conn_01x04

Commit message: start pcb
Parts:
- added IC1: TB67H451FNG,EL, ComponentSearch:SOIC127P600X170-9N, symbol ComponentSearch:TB67H451FNG,EL
- added M1: Motor_DC, Connector_Phoenix_MSTB:PhoenixContact_MSTBA_2,5_2-G-5,08_1x02_P5.08mm_Horizontal, symbol Motor:Motor_DC
- added R1, R2: 10KOhm, Resistor_SMD:R_0805_2012Metric, symbol Device:R
- added SW1, SW2: SW_Push, Button_Switch_THT:SW_PUSH_6mm_H7.3mm, symbol Switch:SW_Push
- J1: renamed from J2; footprint Connector_PinHeader_2.54mm:PinHeader_1x04_P2.54mm_Vertical -> Connector_PinHeader_2.54mm:PinHeader_2x12_P2.54mm_Vertical
- renumbered IC1 to IC2, J3 to J2, J1 to J3, R1 to R3, R2 to R4, TP2 to TP1, TP1 to TP2
Connections:
- net +3.3V: now also J1.13 (Pin_13), IC1.4 (VREF), R1.2, R2.2
- net +5V: now also J1.15 (Pin_15)
- net ARGB: now also IC2.27 (IO0); no longer IC2.26 (IO45)
- net GND: now also J1.14 (Pin_14), J1.16 (Pin_16), IC1.1 (GND), IC1.7 (RS), IC1.9 (EP), SW1.2, SW2.2
- net H.L8: now also IC2.30 (IO37); no longer IC2.27 (IO0)
- net H.R0: now also J1.19 (Pin_19); no longer J1.17 (Pin_17)
- net H.R1: now also J1.20 (Pin_20); no longer J1.18 (Pin_18)
- net H.R2: now also J1.21 (Pin_21); no longer J1.19 (Pin_19)
- net H.R3: now also J1.22 (Pin_22); no longer J1.20 (Pin_20)
- net H.R4: now also J1.23 (Pin_23); no longer J1.21 (Pin_21)
- net H.R5: now also J1.24 (Pin_24); no longer J1.22 (Pin_22)
- net I2C/SMclk: now also J1.18 (Pin_18); no longer J1.16 (Pin_16)
- net I2C/SMdata: now also J1.17 (Pin_17); no longer J1.15 (Pin_15)
- net Button2: now reaches IC2.28 (IO35)
- net Button2: now also R2.1, SW2.1
- net Button1: now reaches IC2.29 (IO36)
- net Button1: now also R1.1, SW1.1
- net H.R6 renamed Motor_in1
- net Motor_in1: now also IC1.2 (IN2); no longer J1.23 (Pin_23)
- net H.R7 renamed Motor_in2
- net Motor_in2: now also IC1.3 (IN1); no longer J1.24 (Pin_24)
- new net: IC1.6 (OUT1), M1.2 (-)
- new net: IC1.8 (OUT2), M1.1 (+)
- new net 5V-24V: IC1.5 (VM)
- no-connect marks 4 -> 1
Other:
- sheet USB ports: added none; removed FAULT_IN
- note added: "Buttons"
- note added: "IO37,36,35 have some functions for the psram that this chip does not have."
- note added: "IO45 cant be high on boot"
- note added: "Motor driver"
- note added: "Uart for logging and programing"
- note removed: "Uart for loging and programming"

Commit message: done for the day
Parts:
- removed J1: Conn_02x12_Top_Bottom, Connector_PinHeader_2.54mm:PinHeader_2x12_P2.54mm_Vertical, symbol Connector_Generic:Conn_02x12_Top_Bottom
- added J1: Conn_02x12_Odd_Even, Connector_PinHeader_2.54mm:PinHeader_2x12_P2.54mm_Vertical, symbol Connector_Generic:Conn_02x12_Odd_Even
Connections:
- net +3.3V: now also J1.1 (Pin_1), J1.2 (Pin_2)
- net +5V: now also J1.5 (Pin_5), J1.6 (Pin_6)
- net CW: now also IC2.16 (IO46); no longer IC2.18 (IO10)
- net G: now also IC2.18 (IO10); no longer IC2.16 (IO46)
- net GND: now also J1.3 (Pin_3), J1.4 (Pin_4), J1.8 (Pin_8)
- net H.L0: now also J1.7 (Pin_7)
- net H.L1: now also J1.9 (Pin_9)
- net H.L2: now also J1.11 (Pin_11)
- net H.L3: now also J1.13 (Pin_13)
- net H.L4: now also J1.15 (Pin_15)
- net H.L5: now also J1.17 (Pin_17)
- net H.L6: now also J1.19 (Pin_19)
- net H.L7: now also J1.21 (Pin_21)
- net H.L8: now also J1.23 (Pin_23)
- net H.R0: now also J1.14 (Pin_14)
- net H.R1: now also J1.16 (Pin_16)
- net H.R2: now also J1.18 (Pin_18)
- net H.R3: now also J1.20 (Pin_20)
- net H.R4: now also J1.22 (Pin_22)
- net H.R5: now also J1.24 (Pin_24)
- net I2C/SMclk: now also J1.12 (Pin_12)
- net I2C/SMdata: now also J1.10 (Pin_10)
- net R: now also IC2.19 (IO11); no longer IC2.15 (IO3)
- net RX0: now also J2.3 (Pin_3); no longer J2.4 (Pin_4)
- net TX0: now also J2.4 (Pin_4); no longer J2.3 (Pin_3)
- net WW: now also IC2.15 (IO3); no longer IC2.19 (IO11)
- net at IC1.6 (OUT1): now also M1.1 (+); no longer M1.2 (-)
- net at IC1.8 (OUT2): now also M1.2 (-); no longer M1.1 (+)
Other:
- moved on the sheet: M1

Commit message: posible V0.1
Parts:
- added H1, H4: MountingHole, MountingHole:MountingHole_4.3mm_M4, symbol Mechanical:MountingHole
- added H2, H3: MountingHole_Pad, MountingHole:MountingHole_4.3mm_M4_Pad, symbol Mechanical:MountingHole_Pad
- added TP3: Power, TestPoint:TestPoint_Loop_D2.60mm_Drill1.4mm_Beaded, symbol Connector:TestPoint
- added TP4: 3.3V, TestPoint:TestPoint_Loop_D2.60mm_Drill1.4mm_Beaded, symbol Connector:TestPoint
- added TP5: 5V, TestPoint:TestPoint_Loop_D2.60mm_Drill1.4mm_Beaded, symbol Connector:TestPoint
Connections:
- net +3.3V: now also J1.5 (Pin_5), J1.6 (Pin_6), TP4.1; no longer J1.1 (Pin_1), J1.2 (Pin_2)
- net +5V: now also J1.1 (Pin_1), J1.2 (Pin_2), TP5.1; no longer J1.5 (Pin_5), J1.6 (Pin_6)
- net 5V-24V: now also TP3.1
- net B: now also IC2.20 (IO12); no longer IC2.17 (IO9)
- net CW: now also IC2.19 (IO11); no longer IC2.16 (IO46)
- net G: now also IC2.21 (IO13); no longer IC2.18 (IO10)
- net GND: now also H2.1, H3.1
- net LD2410_I/O: now also IC2.17 (IO9); no longer IC2.22 (IO14)
- net Motor_in1: now also IC2.12 (IO8); no longer IC2.11 (IO18)
- net Motor_in2: now also IC2.11 (IO18); no longer IC2.12 (IO8)
- net R: now also IC2.22 (IO14); no longer IC2.19 (IO11)
- net RX: now also IC2.16 (IO46); no longer IC2.21 (IO13)
- net TX: now also IC2.15 (IO3); no longer IC2.20 (IO12)
- net WW: now also IC2.18 (IO10); no longer IC2.15 (IO3)
Other:
- sheet I2C Connectors ports: added I2C/SMclk, I2C/SMdata; removed none

Commit message: v0.1
Other:
- note added: "IO35->42 are not gpio by default"
- note added: "IO37,36,35 have some functions for the psram that this chip does not have. may cause issues."
- note added: "Mounting holes"
- note added: "Power Test Points"
- note removed: "IO37,36,35 have some functions for the psram that this chip does not have."
- moved on the sheet: H1, H2, H3, H4, TP3, TP4, TP5
