File: KiCad Schematics and pcb/ESPHome AIO.kicad_sch (KiCad schematic)
At the start: 21 parts, among them IC1 TB67H451FNG,EL, IC2 ESP32-S3-WROOM-1-N8, J1 Conn_02x12_Odd_Even, J2 Conn_01x04, J3 Conn_01x05, M1 Screw_Terminal_01x02, SW1 SW_Push, SW2 SW_Push

Commit message: V0.2 maybe
Parts:
- added C14: 100nF, Capacitor_SMD:C_0805_2012Metric, symbol Device:C_Small
- added R39: 10K, Resistor_SMD:R_0805_2012Metric, symbol Device:R
- added SW7: SW_Push, Button_Switch_THT:SW_PUSH_6mm_H7.3mm, symbol Switch:SW_Push
Connections:
- net +3.3V: now also R39.2; no longer IC2.3 (EN)
- net GND: now also C14.1, SW7.2
- new net EN: C14.2, IC2.3 (EN), R39.1, SW7.1
Changed lines of the file:
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@@
   (junction (at 222.25 140.97) (diameter 0) (color 0 0 0 0)
   )
-  (junction (at 144.78 33.02) (diameter 0) (color 0 0 0 0)
-  )
   (junction (at 26.67 60.96) (diameter 0) (color 0 0 0 0)
   )
   (junction (at 33.02 185.42) (diameter 0) (color 0 0 0 0)
+  )
+  (junction (at 39.37 110.49) (diameter 0) (color 0 0 0 0)
+  )
+  (junction (at 24.13 110.49) (diameter 0) (color 0 0 0 0)
   )
   (junction (at 222.25 118.11) (diameter 0) (color 0 0 0 0)
@@
     (stroke (width 0) (type default))
   )
+  (wire (pts (xy 38.1 110.49) (xy 39.37 110.49))
+    (stroke (width 0) (type default))
+  )
   (wire (pts (xy 52.07 93.98) (xy 63.5 93.98))
     (stroke (width 0) (type default))
@@
     (stroke (width 0) (type default))
   )
+  (wire (pts (xy 142.875 35.56) (xy 146.05 35.56))
+    (stroke (width 0) (type default))
+  )
   (wire (pts (xy 199.39 58.42) (xy 208.28 58.42))
     (stroke (width 0) (type default))
@@
     (stroke (width 0) (type default))
   )
-  (wire (pts (xy 199.39 60.96) (xy 205.74 60.96))
+  (wire (pts (xy 199.39 60.96) (xy 208.28 60.96))
     (stroke (width 0) (type default))
   )
@@
     (stroke (width 0) (type default))
   )
+  (wire (pts (xy 24.13 110.49) (xy 24.13 103.505))
+    (stroke (width 0) (type default))
+  )
   (wire (pts (xy 52.07 96.52) (xy 63.5 96.52))
     (stroke (width 0) (type default))
@@
     (stroke (width 0) (type default))
   )
-  (wire (pts (xy 143.51 33.02) (xy 144.78 33.02))
-    (stroke (width 0) (type default))
-  )
   (wire (pts (xy 209.55 138.43) (xy 209.55 128.27))
     (stroke (width 0) (type default))
@@
     (stroke (width 0) (type default))
   )
+  (wire (pts (xy 30.48 118.745) (xy 24.13 118.745))
+    (stroke (width 0) (type default))
+  )
   (wire (pts (xy 60.96 100.33) (xy 60.96 99.06))
     (stroke (width 0) (type default))
@@
     (stroke (width 0) (type default))
   )
-  (wire (pts (xy 146.05 35.56) (xy 144.78 35.56))
-    (stroke (width 0) (type default))
-  )
   (wire (pts (xy 233.68 44.45) (xy 243.84 44.45))
     (stroke (width 0) (type default))
@@
     (stroke (width 0) (type default))
   )
+  (wire (pts (xy 44.45 112.395) (xy 44.45 110.49))
+    (stroke (width 0) (type default))
+  )
   (wire (pts (xy 173.99 71.12) (xy 173.99 85.09))
     (stroke (width 0) (type default))
@@
     (stroke (width 0) (type default))
   )
+  (wire (pts (xy 17.145 110.49) (xy 24.13 110.49))
+    (stroke (width 0) (type default))
+  )
   (bus (pts (xy 231.14 34.29) (xy 231.14 36.83))
     (stroke (width 0) (type default))
@@
     (stroke (width 0) (type default))
   )
+  (wire (pts (xy 24.13 118.745) (xy 24.13 110.49))
+    (stroke (width 0) (type default))
+  )
   (wire (pts (xy 77.47 54.61) (xy 92.71 54.61))
     (stroke (width 0) (type default))
@@
     (stroke (width 0) (type default))
   )
-  (wire (pts (xy 144.78 35.56) (xy 144.78 33.02))
-    (stroke (width 0) (type default))
-  )
   (wire (pts (xy 77.47 27.94) (xy 93.98 27.94))
     (stroke (width 0) (type default))
@@
     (stroke (width 0) (type default))
   )
+  (wire (pts (xy 35.56 118.745) (xy 39.37 118.745))
+    (stroke (width 0) (type default))
+  )
   (wire (pts (xy 110.49 99.06) (xy 110.49 101.6))
     (stroke (width 0) (type default))
@@
     (stroke (width 0) (type default))
   )
-  (wire (pts (xy 144.78 33.02) (xy 146.05 33.02))
+  (wire (pts (xy 143.51 33.02) (xy 146.05 33.02))
     (stroke (width 0) (type default))
   )
@@
     (stroke (width 0) (type default))
   )
+  (wire (pts (xy 39.37 110.49) (xy 44.45 110.49))
+    (stroke (width 0) (type default))
+  )
   (wire (pts (xy 222.25 140.97) (xy 236.22 140.97))
     (stroke (width 0) (type default))
@@
     (stroke (width 0) (type default))
   )
+  (wire (pts (xy 24.13 110.49) (xy 27.94 110.49))
+    (stroke (width 0) (type default))
+  )
   (wire (pts (xy 236.22 31.75) (xy 243.84 31.75))
     (stroke (width 0) (type default))
   )
   (wire (pts (xy 27.94 185.42) (xy 33.02 185.42))
+    (stroke (width 0) (type default))
+  )
+  (wire (pts (xy 39.37 118.745) (xy 39.37 110.49))
     (stroke (width 0) (type default))
   )
@@
     (fill (type none))
   )
-  (rectangle (start 13.97 39.37) (end 49.53 96.52)
+  (rectangle (start 13.97 39.37) (end 49.53 127.635)
     (stroke (width 0) (type dash))
     (fill (type none))
@@
     (effects (font (size 1.27 1.27)) (justify left bottom))
   )
+  (label "EN" (at 17.145 110.49 0) (fields_autoplaced)
+    (effects (font (size 1.27 1.27)) (justify left bottom))
+  )
   (label "RX0" (at 205.74 38.1 180) (fields_autoplaced)
     (effects (font (size 1.27 1.27)) (justify right bottom))
@@
     (effects (font (size 1.27 1.27)) (justify right bottom))
   )
-  (label "ARGB" (at 205.74 60.96 180) (fields_autoplaced)
+  (label "ARGB" (at 208.28 60.96 180) (fields_autoplaced)
     (effects (font (size 1.27 1.27)) (justify right bottom))
   )
@@
   )
   (label "LD2410_I{slash}O" (at 251.46 149.86 0) (fields_autoplaced)
+    (effects (font (size 1.27 1.27)) (justify left bottom))
+  )
+  (label "EN" (at 142.875 35.56 0) (fields_autoplaced)
     (effects (font (size 1.27 1.27)) (justify left bottom))
   )
@@
         (path "/5cdf3b4f-d143-42e3-ac6f-eec5265de1fa"
           (reference "#PWR06") (unit 1)
+        )
+      )
+    )
+  )
+  (symbol (lib_id "Device:R") (at 24.13 99.695 180) (unit 1)
+    (in_bom yes) (on_board yes) (dnp no) (fields_autoplaced)
+    (property "Reference" "R39" (at 26.67 98.425 0)
+      (effects (font (size 1.27 1.27)) (justify right))
+    )
+    (property "Value" "10K" (at 26.67 100.965 0)
+      (effects (font (size 1.27 1.27)) (justify right))
+    )
+    (property "Footprint" "Resistor_SMD:R_0805_2012Metric" (at 25.908 99.695 90)
+      (effects (font (size 1.27 1.27)) hide)
+    )
+    (property "Datasheet" "~" (at 24.13 99.695 0)
+      (effects (font (size 1.27 1.27)) hide)
+    )
+    (property "LCSC" "C17414" (at 24.13 99.695 0)
+      (effects (font (size 1.27 1.27)) hide)
+    )
+    (pin "2")
+    (pin "1")
+    (instances
+      (project "ESPHome AIO"
+        (path "/5cdf3b4f-d143-42e3-ac6f-eec5265de1fa"
+          (reference "R39") (unit 1)
         )
       )
@@
     )
   )
+  (symbol (lib_id "Switch:SW_Push") (at 33.02 110.49 0) (unit 1)
+    (in_bom yes) (on_board yes) (dnp no)
+    (property "Reference" "SW7" (at 33.02 113.03 0)
+      (effects (font (size 1.27 1.27)))
+    )
+    (property "Value" "SW_Push" (at 33.02 115.57 0)
+      (effects (font (size 1.27 1.27)))
+    )
+    (property "Footprint" "Button_Switch_THT:SW_PUSH_6mm_H7.3mm" (at 33.02 105.41 0)
+      (effects (font (size 1.27 1.27)) hide)
+    )
+    (property "Datasheet" "~" (at 33.02 105.41 0)
+      (effects (font (size 1.27 1.27)) hide)
+    )
+    (property "LCSC" "C7463311" (at 33.02 110.49 0)
+      (effects (font (size 1.27 1.27)) hide)
+    )
+    (pin "2")
+    (pin "1")
+    (instances
+      (project "ESPHome AIO"
+        (path "/5cdf3b4f-d143-42e3-ac6f-eec5265de1fa"
+          (reference "SW7") (unit 1)
+        )
+      )
+    )
+  )
+  (symbol (lib_id "power:+3.3V") (at 24.13 95.885 0) (unit 1)
+    (in_bom yes) (on_board yes) (dnp no) (fields_autoplaced)
+    (property "Reference" "#PWR050" (at 24.13 99.695 0)
+      (effects (font (size 1.27 1.27)) hide)
+    )
+    (property "Value" "+3.3V" (at 24.13 90.805 0)
+      (effects (font (size 1.27 1.27)))
+    )
+    (property "Footprint" "" (at 24.13 95.885 0)
+      (effects (font (size 1.27 1.27)) hide)
+    )
+    (property "Datasheet" "" (at 24.13 95.885 0)
+      (effects (font (size 1.27 1.27)) hide)
+    )
+    (pin "1")
+    (instances
+      (project "ESPHome AIO"
+        (path "/5cdf3b4f-d143-42e3-ac6f-eec5265de1fa"
+          (reference "#PWR050") (unit 1)
+        )
+      )
+    )
+  )
   (symbol (lib_id "ComponentSearch:TB67H451FNG,EL") (at 63.5 91.44 0) (unit 1)
     (in_bom yes) (on_board yes) (dnp no) (fields_autoplaced)
@@
     )
   )
+  (symbol (lib_id "power:GND") (at 44.45 112.395 0) (unit 1)
+    (in_bom yes) (on_board yes) (dnp no) (fields_autoplaced)
+    (property "Reference" "#PWR052" (at 44.45 118.745 0)
+      (effects (font (size 1.27 1.27)) hide)
+    )
+    (property "Value" "GND" (at 44.45 117.475 0)
+      (effects (font (size 1.27 1.27)))
+    )
+    (property "Footprint" "" (at 44.45 112.395 0)
+      (effects (font (size 1.27 1.27)) hide)
+    )
+    (property "Datasheet" "" (at 44.45 112.395 0)
+      (effects (font (size 1.27 1.27)) hide)
+    )
+    (pin "1")
+    (instances
+      (project "ESPHome AIO"
+        (path "/5cdf3b4f-d143-42e3-ac6f-eec5265de1fa"
+          (reference "#PWR052") (unit 1)
+        )
+      )
+    )
+  )
   (symbol (lib_id "power:+3.3V") (at 139.7 31.75 180) (unit 1)
     (in_bom yes) (on_board yes) (dnp no) (fields_autoplaced)
@@
         )
       )
+    )
+  )
+  (symbol (lib_id "Device:C_Small") (at 33.02 118.745 270) (unit 1)
+    (in_bom yes) (on_board yes) (dnp no)
+    (property "Reference" "C14" (at 33.02 121.92 90)
+      (effects (font (size 1.27 1.27)))
+    )
+    (property "Value" "100nF" (at 33.02 124.46 90)
+      (effects (font (size 1.27 1.27)))
+    )
+    (property "Footprint" "Capacitor_SMD:C_0805_2012Metric" (at 33.02 118.745 0)
+      (effects (font (size 1.27 1.27)) hide)
+    )
+    (property "Datasheet" "~" (at 33.02 118.745 0)
+      (effects (font (size 1.27 1.27)) hide)
+    )
+    (property "LCSC" "" (at 33.02 118.745 0)
+      (effects (font (size 1.27 1.27)) hide)
+    )
+    (pin "1")
+    (pin "2")
+    (instances
+      (project "ESPHome AIO"
+        (path "/5cdf3b4f-d143-42e3-ac6f-eec5265de1fa"
+          (reference "C14") (unit 1)
+        )
+      )

Commit message: V0.2 wip
Parts:
- added JP4: Jumper_2_Open, symbol Jumper:Jumper_2_Open
Connections:
- net ARGB: now also JP4.1 (A)
- net GND: now also JP4.2 (B)
- net Motor_in1: now also IC1.3 (IN1), IC2.11 (IO18); no longer IC1.2 (IN2), IC2.12 (IO8)
- net Motor_in2: now also IC1.2 (IN2), IC2.12 (IO8); no longer IC1.3 (IN1), IC2.11 (IO18)
Other:
- sheet Power ports: added VBUS; removed none
- sheet USB ports: added VBUS; removed none
- note added: "Boot Jumper"

Commit message: 0.2
Parts:
- added D8: LED, LED_SMD:LED_0805_2012Metric, symbol Device:LED
- added R40: 10K, Resistor_SMD:R_0805_2012Metric, symbol Device:R
- JP4: footprint (none) -> Connector_PinHeader_2.54mm:PinHeader_1x02_P2.54mm_Vertical
Connections:
- net 5V-24V: now also D8.2 (A)
- net GND: now also R40.2
- new net: D8.1 (K), R40.1
Other:
- note added: "Power LED"
