File: KiCad Schematics and pcb/USB.kicad_sch (KiCad schematic)
At the start: 19 parts, among them IC3 TPS25730DREFR, J6 USB_C_Receptacle_USB2.0_16P, U1 TVS2200DRV

Commit message: start pcb
Parts:
- IC4: renamed from IC3; footprint TPS25730DREFR -> ComponentSearch:TPS25730DREFR
- renumbered J6 to J7, R10 to R14, R11 to R15, R12 to R16
Connections:
- net GND: now also IC4.34 (GND), IC4.35 (GND), IC4.44 (GND); no longer IC4.34,35,44 (GND)
- net USB_POWER: now reaches C1.2, C2.2, C4.2, D1.2 (A)
- net USB_POWER: now also IC4.20 (PPHV), IC4.21 (PPHV), IC4.22 (PPHV), IC4.41 (PPHV); no longer IC4.20,21,22,41 (PPHV)
- net VBUS: now reaches C5.1, C7.1, C9.1, J7.A4 (VBUS), J7.A9 (VBUS), J7.B4 (VBUS), J7.B9 (VBUS), TP5.1, U1.4 (IN), U1.5 (IN), U1.6 (IN)
- net VBUS: now also IC4.23 (VBUS_IN), IC4.24 (VBUS_IN), IC4.25 (VBUS_IN), IC4.32 (VBUS), IC4.33 (VBUS), IC4.42 (VBUS_IN), IC4.43 (VBUS); no longer IC4.23,24,25.42 (VBUS_IN), IC4.33,32,43 (VBUS)
- net DBG_ACC: no longer names the net of IC4.10 (DBG_ACC)
- net FAULT_IN: no longer names the net of IC4.18 (~{FAULT_IN}), R14.2
- net PLUG_FLIP: no longer names the net of IC4.13 (PLUG_FLIP)
- no-connect marks 4 -> 6
Other:
- removed sheet Led Driver2
- removed sheet Led Driver3
- note added: "Signal LEDs for usb c debugging"

Commit message: done for the day
Parts:
- removed TP3: CC2, TestPoint:TestPoint_Loop_D2.60mm_Drill1.4mm_Beaded, symbol Connector:TestPoint
- removed TP4: CC1, TestPoint:TestPoint_Loop_D2.60mm_Drill1.4mm_Beaded, symbol Connector:TestPoint
Changed lines of the file:
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@@
   (junction (at 166.37 40.64) (diameter 0) (color 0 0 0 0)
   )
-  (junction (at 175.26 66.04) (diameter 0) (color 0 0 0 0)
-  )
   (junction (at 39.37 104.14) (diameter 0) (color 0 0 0 0)
   )
@@
   )
   (junction (at 109.22 88.9) (diameter 0) (color 0 0 0 0)
-  )
-  (junction (at 175.26 63.5) (diameter 0) (color 0 0 0 0)
   )
   (junction (at 210.82 16.51) (diameter 0) (color 0 0 0 0)
@@
     (stroke (width 0) (type default))
   )
-  (wire (pts (xy 175.26 66.04) (xy 189.23 66.04))
-    (stroke (width 0) (type default))
-  )
   (wire (pts (xy 106.68 99.06) (xy 109.22 99.06))
     (stroke (width 0) (type default))
@@
     (stroke (width 0) (type default))
   )
-  (wire (pts (xy 106.68 63.5) (xy 175.26 63.5))
+  (wire (pts (xy 106.68 63.5) (xy 201.93 63.5))
     (stroke (width 0) (type default))
   )
@@
     (stroke (width 0) (type default))
   )
-  (wire (pts (xy 175.26 63.5) (xy 201.93 63.5))
-    (stroke (width 0) (type default))
-  )
   (wire (pts (xy 40.64 66.04) (xy 49.53 66.04))
     (stroke (width 0) (type default))
@@
     (stroke (width 0) (type default))
   )
-  (wire (pts (xy 106.68 66.04) (xy 175.26 66.04))
+  (wire (pts (xy 106.68 66.04) (xy 189.23 66.04))
     (stroke (width 0) (type default))
   )
@@
         (path "/5cdf3b4f-d143-42e3-ac6f-eec5265de1fa/f403fb1f-6c3a-4b91-96f2-7610e89c4ca7"
           (reference "C2") (unit 1)
-        )
-      )
-    )
-  )
-  (symbol (lib_id "Connector:TestPoint") (at 175.26 66.04 180) (unit 1)
-    (in_bom yes) (on_board yes) (dnp no) (fields_autoplaced)
-    (property "Reference" "TP4" (at 177.8 68.072 0)
-      (effects (font (size 1.27 1.27)) (justify right))
-    )
-    (property "Value" "CC1" (at 177.8 70.612 0)
-      (effects (font (size 1.27 1.27)) (justify right))
-    )
-    (property "Footprint" "TestPoint:TestPoint_Loop_D2.60mm_Drill1.4mm_Beaded" (at 170.18 66.04 0)
-      (effects (font (size 1.27 1.27)) hide)
-    )
-    (property "Datasheet" "~" (at 170.18 66.04 0)
-      (effects (font (size 1.27 1.27)) hide)
-    )
-    (pin "1")
-    (instances
-      (project "ESPHome AIO"
-        (path "/5cdf3b4f-d143-42e3-ac6f-eec5265de1fa/f403fb1f-6c3a-4b91-96f2-7610e89c4ca7"
-          (reference "TP4") (unit 1)
         )
       )
@@
         )
       )
-    )
-  )
-  (symbol (lib_id "Connector:TestPoint") (at 175.26 63.5 0) (unit 1)
-    (in_bom yes) (on_board yes) (dnp no) (fields_autoplaced)
-    (property "Reference" "TP3" (at 177.8 58.928 0)
-      (effects (font (size 1.27 1.27)) (justify left))
-    )
-    (property "Value" "CC2" (at 177.8 61.468 0)
-      (effects (font (size 1.27 1.27)) (justify left))
-    )
-    (property "Footprint" "TestPoint:TestPoint_Loop_D2.60mm_Drill1.4mm_Beaded" (at 180.34 63.5 0)
-      (effects (font (size 1.27 1.27)) hide)
-    )
-    (property "Datasheet" "~" (at 180.34 63.5 0)
-      (effects (font (size 1.27 1.27)) hide)
-    )
-    (pin "1")
-    (instances
-      (project "ESPHome AIO"
-        (path "/5cdf3b4f-d143-42e3-ac6f-eec5265de1fa/f403fb1f-6c3a-4b91-96f2-7610e89c4ca7"
-          (reference "TP3") (unit 1)
-        )
-      )

Commit message: posible V0.1
Parts:
- removed TP5: VBUS, TestPoint:TestPoint_Loop_D2.60mm_Drill1.4mm_Beaded, symbol Connector:TestPoint
Other:
- removed sheet Led Driver4
Changed lines of the file:
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@@
   (junction (at 49.53 66.04) (diameter 0) (color 0 0 0 0)
-  )
-  (junction (at 218.44 21.59) (diameter 0) (color 0 0 0 0)
   )
   (junction (at 109.22 104.14) (diameter 0) (color 0 0 0 0)
@@
     (stroke (width 0) (type default))
   )
-  (wire (pts (xy 205.74 114.3) (xy 210.82 114.3))
-    (stroke (width 0) (type default))
-  )
   (wire (pts (xy 205.74 43.18) (xy 205.74 40.64))
     (stroke (width 0) (type default))
@@
     (stroke (width 0) (type default))
   )
-  (wire (pts (xy 248.92 130.81) (xy 254 130.81))
-    (stroke (width 0) (type default))
-  )
   (wire (pts (xy 189.23 66.04) (xy 228.6 66.04))
     (stroke (width 0) (type default))
@@
     (stroke (width 0) (type default))
   )
+  (wire (pts (xy 209.55 113.03) (xy 209.55 114.3))
+    (stroke (width 0) (type default))
+  )
   (wire (pts (xy 135.89 31.75) (xy 135.89 50.8))
     (stroke (width 0) (type default))
@@
     (stroke (width 0) (type default))
   )
-  (wire (pts (xy 248.92 128.27) (xy 248.92 130.81))
-    (stroke (width 0) (type default))
-  )
   (wire (pts (xy 49.53 72.39) (xy 57.15 72.39))
     (stroke (width 0) (type default))
@@
     (stroke (width 0) (type default))
   )
+  (wire (pts (xy 209.55 114.3) (xy 214.63 114.3))
+    (stroke (width 0) (type default))
+  )
   (wire (pts (xy 106.68 104.14) (xy 109.22 104.14))
     (stroke (width 0) (type default))
@@
     (stroke (width 0) (type default))
   )
+  (wire (pts (xy 204.47 116.84) (xy 214.63 116.84))
+    (stroke (width 0) (type default))
+  )
   (wire (pts (xy 227.33 55.88) (xy 228.6 55.88))
     (stroke (width 0) (type default))
@@
     (stroke (width 0) (type default))
   )
-  (wire (pts (xy 218.44 21.59) (xy 218.44 16.51))
+  (wire (pts (xy 218.44 16.51) (xy 218.44 71.12))
     (stroke (width 0) (type default))
   )
@@
     (stroke (width 0) (type default))
   )
-  (wire (pts (xy 205.74 111.76) (xy 205.74 114.3))
-    (stroke (width 0) (type default))
-  )
-  (wire (pts (xy 195.58 116.84) (xy 210.82 116.84))
-    (stroke (width 0) (type default))
-  )
   (wire (pts (xy 201.93 33.02) (xy 201.93 40.64))
     (stroke (width 0) (type default))
@@
     (stroke (width 0) (type default))
   )
-  (wire (pts (xy 218.44 71.12) (xy 218.44 21.59))
-    (stroke (width 0) (type default))
-  )
   (wire (pts (xy 106.68 96.52) (xy 109.22 96.52))
-    (stroke (width 0) (type default))
-  )
-  (wire (pts (xy 243.84 133.35) (xy 254 133.35))
     (stroke (width 0) (type default))
   )
@@
     (effects (font (size 1.27 1.27)) (justify left bottom))
   )
+  (label "SINK_EN" (at 204.47 116.84 0) (fields_autoplaced)
+    (effects (font (size 1.27 1.27)) (justify left bottom))
+  )
   (label "USB_POWER" (at 60.96 60.96 180) (fields_autoplaced)
     (effects (font (size 1.27 1.27)) (justify right bottom))
@@
   (label "CAP_MIS" (at 115.57 71.12 180) (fields_autoplaced)
     (effects (font (size 1.27 1.27)) (justify right bottom))
-  )
-  (label "SINK_EN" (at 243.84 133.35 0) (fields_autoplaced)
-    (effects (font (size 1.27 1.27)) (justify left bottom))
-  )
-  (label "PLUG_EVENT" (at 195.58 116.84 0) (fields_autoplaced)
-    (effects (font (size 1.27 1.27)) (justify left bottom))
   )
   (label "PLUG_EVENT" (at 48.26 78.74 0) (fields_autoplaced)
@@
         (path "/5cdf3b4f-d143-42e3-ac6f-eec5265de1fa/f403fb1f-6c3a-4b91-96f2-7610e89c4ca7"
           (reference "#PWR052") (unit 1)
-        )
-      )
-    )
-  )
-  (symbol (lib_id "ComponentSearch:LDO_3V3") (at 205.74 111.76 0) (unit 1)
-    (in_bom yes) (on_board yes) (dnp no) (fields_autoplaced)
-    (property "Reference" "#PWR059" (at 205.74 115.57 0)
-      (effects (font (size 1.27 1.27)) hide)
-    )
-    (property "Value" "LDO_3V3" (at 205.74 106.68 0)
-      (effects (font (size 1.27 1.27)))
-    )
-    (property "Footprint" "" (at 205.74 111.76 0)
-      (effects (font (size 1.27 1.27)) hide)
-    )
-    (property "Datasheet" "" (at 205.74 111.76 0)
-      (effects (font (size 1.27 1.27)) hide)
-    )
-    (pin "1")
-    (instances
-      (project "ESPHome AIO"
-        (path "/5cdf3b4f-d143-42e3-ac6f-eec5265de1fa/f403fb1f-6c3a-4b91-96f2-7610e89c4ca7"
-          (reference "#PWR059") (unit 1)
         )
       )
@@
     )
   )
-  (symbol (lib_id "Connector:TestPoint") (at 218.44 21.59 270) (unit 1)
-    (in_bom yes) (on_board yes) (dnp no) (fields_autoplaced)
-    (property "Reference" "TP5" (at 223.52 20.32 90)
-      (effects (font (size 1.27 1.27)) (justify left))
-    )
-    (property "Value" "VBUS" (at 223.52 22.86 90)
-      (effects (font (size 1.27 1.27)) (justify left))
-    )
-    (property "Footprint" "TestPoint:TestPoint_Loop_D2.60mm_Drill1.4mm_Beaded" (at 218.44 26.67 0)
-      (effects (font (size 1.27 1.27)) hide)
-    )
-    (property "Datasheet" "~" (at 218.44 26.67 0)
-      (effects (font (size 1.27 1.27)) hide)
-    )
-    (pin "1")
-    (instances
-      (project "ESPHome AIO"
-        (path "/5cdf3b4f-d143-42e3-ac6f-eec5265de1fa/f403fb1f-6c3a-4b91-96f2-7610e89c4ca7"
-          (reference "TP5") (unit 1)
-        )
-      )
-    )
-  )
   (symbol (lib_id "power:GND") (at 166.37 52.07 0) (unit 1)
     (in_bom yes) (on_board yes) (dnp no) (fields_autoplaced)
@@
         (path "/5cdf3b4f-d143-42e3-ac6f-eec5265de1fa/f403fb1f-6c3a-4b91-96f2-7610e89c4ca7"
           (reference "D1") (unit 1)
+        )
+      )
+    )
+  )
+  (symbol (lib_id "ComponentSearch:LDO_3V3") (at 209.55 113.03 0) (unit 1)
+    (in_bom yes) (on_board yes) (dnp no) (fields_autoplaced)
+    (property "Reference" "#PWR059" (at 209.55 116.84 0)
+      (effects (font (size 1.27 1.27)) hide)
+    )
+    (property "Value" "LDO_3V3" (at 209.55 107.95 0)
+      (effects (font (size 1.27 1.27)))
+    )
+    (property "Footprint" "" (at 209.55 113.03 0)
+      (effects (font (size 1.27 1.27)) hide)
+    )
+    (property "Datasheet" "" (at 209.55 113.03 0)
+      (effects (font (size 1.27 1.27)) hide)
+    )
+    (pin "1")
+    (instances
+      (project "ESPHome AIO"
+        (path "/5cdf3b4f-d143-42e3-ac6f-eec5265de1fa/f403fb1f-6c3a-4b91-96f2-7610e89c4ca7"
+          (reference "#PWR059") (unit 1)
         )
       )
@@
         (path "/5cdf3b4f-d143-42e3-ac6f-eec5265de1fa/f403fb1f-6c3a-4b91-96f2-7610e89c4ca7"
           (reference "C7") (unit 1)
-        )
-      )
-    )
-  )
-  (symbol (lib_id "ComponentSearch:LDO_3V3") (at 248.92 128.27 0) (unit 1)
-    (in_bom yes) (on_board yes) (dnp no) (fields_autoplaced)
-    (property "Reference" "#PWR061" (at 248.92 132.08 0)
-      (effects (font (size 1.27 1.27)) hide)
-    )
-    (property "Value" "LDO_3V3" (at 248.92 123.19 0)
-      (effects (font (size 1.27 1.27)))
-    )
-    (property "Footprint" "" (at 248.92 128.27 0)
-      (effects (font (size 1.27 1.27)) hide)
-    )
-    (property "Datasheet" "" (at 248.92 128.27 0)
-      (effects (font (size 1.27 1.27)) hide)
-    )
-    (pin "1")
-    (instances
-      (project "ESPHome AIO"
-        (path "/5cdf3b4f-d143-42e3-ac6f-eec5265de1fa/f403fb1f-6c3a-4b91-96f2-7610e89c4ca7"
-          (reference "#PWR061") (unit 1)
         )
       )
@@
           (reference "R16") (unit 1)
         )
-      )
-    )
-  )
-  (sheet (at 210.82 111.76) (size 12.7 7.62) (fields_autoplaced)
-    (stroke (width 0.1524) (type solid))
-    (fill (color 0 0 0 0.0000))
-    (property "Sheetname" "Led Driver4" (at 210.82 111.0484 0)
-      (effects (font (size 1.27 1.27)) (justify left bottom))
-    )
-    (property "Sheetfile" "SignalLed.kicad_sch" (at 210.82 119.9646 0)
-      (effects (font (size 1.27 1.27)) (justify left top))
-    )
-    (pin "GPIO" input (at 210.82 116.84 180)
-      (effects (font (size 1.27 1.27)) (justify left))
-    )
-    (pin "V+" input (at 210.82 114.3 180)
-      (effects (font (size 1.27 1.27)) (justify left))
-    )
-    (instances
-      (project "ESPHome AIO"
-        (path "/5cdf3b4f-d143-42e3-ac6f-eec5265de1fa/f403fb1f-6c3a-4b91-96f2-7610e89c4ca7" (page "9"))
       )
     )
@@
     )
   )
-  (sheet (at 254 128.27) (size 12.7 7.62) (fields_autoplaced)
+  (sheet (at 214.63 111.76) (size 12.7 7.62) (fields_autoplaced)
     (stroke (width 0.1524) (type solid))
     (fill (color 0 0 0 0.0000))
-    (property "Sheetname" "Led Driver1" (at 254 127.5584 0)
+    (property "Sheetname" "Led Driver1" (at 214.63 111.0484 0)
       (effects (font (size 1.27 1.27)) (justify left bottom))
     )
-    (property "Sheetfile" "SignalLed.kicad_sch" (at 254 136.4746 0)
+    (property "Sheetfile" "SignalLed.kicad_sch" (at 214.63 119.9646 0)
       (effects (font (size 1.27 1.27)) (justify left top))
     )
-    (pin "GPIO" input (at 254 133.35 180)
-      (effects (font (size 1.27 1.27)) (justify left))
-    )
-    (pin "V+" input (at 254 130.81 180)
-      (effects (font (size 1.27 1.27)) (justify left))
-    )
+    (pin "GPIO" input (at 214.63 116.84 180)
+      (effects (font (size 1.27 1.27)) (justify left))
+    )
+    (pin "V+" input (at 214.63 114.3 180)
+      (effects (font (size 1.27 1.27)) (justify left))
+    )

Commit message: v0.1
Other:
- note added: "USB-C connector + decoupling and protection"
- moved on the sheet: C6, C8
Changed lines of the file:
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@@
   (junction (at 49.53 66.04) (diameter 0) (color 0 0 0 0)
   )
+  (junction (at 123.19 76.2) (diameter 0) (color 0 0 0 0)
+  )
   (junction (at 109.22 104.14) (diameter 0) (color 0 0 0 0)
   )
@@
   (junction (at 34.29 60.96) (diameter 0) (color 0 0 0 0)
   )
+  (junction (at 123.19 66.04) (diameter 0) (color 0 0 0 0)
+  )
   (junction (at 44.45 60.96) (diameter 0) (color 0 0 0 0)
   )
@@
   (junction (at 210.82 16.51) (diameter 0) (color 0 0 0 0)
   )
-  (junction (at 189.23 66.04) (diameter 0) (color 0 0 0 0)
-  )
-  (junction (at 201.93 63.5) (diameter 0) (color 0 0 0 0)
-  )
   (junction (at 227.33 52.07) (diameter 0) (color 0 0 0 0)
   )
@@
   )
   (junction (at 251.46 30.48) (diameter 0) (color 0 0 0 0)
+  )
+  (junction (at 134.62 63.5) (diameter 0) (color 0 0 0 0)
   )
   (junction (at 205.74 40.64) (diameter 0) (color 0 0 0 0)
@@
     (stroke (width 0) (type default))
   )
-  (wire (pts (xy 201.93 63.5) (xy 228.6 63.5))
+  (wire (pts (xy 134.62 63.5) (xy 228.6 63.5))
     (stroke (width 0) (type default))
   )
@@
     (stroke (width 0) (type default))
   )
-  (wire (pts (xy 189.23 66.04) (xy 228.6 66.04))
+  (wire (pts (xy 123.19 66.04) (xy 228.6 66.04))
     (stroke (width 0) (type default))
   )
@@
     (stroke (width 0) (type default))
   )
-  (wire (pts (xy 201.93 63.5) (xy 201.93 69.85))
+  (wire (pts (xy 134.62 63.5) (xy 134.62 69.85))
     (stroke (width 0) (type default))
   )
@@
     (stroke (width 0) (type default))
   )
-  (wire (pts (xy 189.23 66.04) (xy 189.23 69.85))
+  (wire (pts (xy 123.19 66.04) (xy 123.19 69.85))
     (stroke (width 0) (type default))
   )
@@
     (stroke (width 0) (type default))
   )
-  (wire (pts (xy 106.68 63.5) (xy 201.93 63.5))
+  (wire (pts (xy 106.68 63.5) (xy 134.62 63.5))
     (stroke (width 0) (type default))
   )
@@
     (stroke (width 0) (type default))
   )
+  (wire (pts (xy 123.19 76.2) (xy 134.62 76.2))
+    (stroke (width 0) (type default))
+  )
   (wire (pts (xy 135.89 50.8) (xy 106.68 50.8))
     (stroke (width 0) (type default))
@@
     (stroke (width 0) (type default))
   )
-  (wire (pts (xy 201.93 74.93) (xy 201.93 76.2))
+  (wire (pts (xy 134.62 74.93) (xy 134.62 76.2))
     (stroke (width 0) (type default))
   )
@@
     (stroke (width 0) (type default))
   )
-  (wire (pts (xy 189.23 74.93) (xy 189.23 76.2))
+  (wire (pts (xy 123.19 77.47) (xy 123.19 76.2))
+    (stroke (width 0) (type default))
+  )
+  (wire (pts (xy 123.19 74.93) (xy 123.19 76.2))
     (stroke (width 0) (type default))
   )
@@
     (stroke (width 0) (type default))
   )
-  (wire (pts (xy 106.68 66.04) (xy 189.23 66.04))
+  (wire (pts (xy 106.68 66.04) (xy 123.19 66.04))
     (stroke (width 0) (type default))
   )
@@
     (stroke (width 0) (type default))
   )
-  (rectangle (start 193.04 101.6) (end 283.21 158.75)
+  (rectangle (start 193.04 101.6) (end 283.21 125.73)
+    (stroke (width 0) (type dash))
+    (fill (type none))
+  )
+  (rectangle (start 180.34 12.7) (end 264.16 83.82)
     (stroke (width 0) (type dash))
     (fill (type none))
@@
     (stroke (width 0) (type dash))
     (fill (type none))
+  )
+  (text "USB-C connector + decoupling and protection" (at 180.34 86.36 0)
+    (effects (font (size 1.27 1.27)) (justify left bottom))
   )
   (text "Signal LEDs for usb c debugging" (at 193.04 101.6 0)
@@
     )
   )
-  (symbol (lib_id "power:GND") (at 189.23 76.2 0) (unit 1)
-    (in_bom yes) (on_board yes) (dnp no) (fields_autoplaced)
-    (property "Reference" "#PWR055" (at 189.23 82.55 0)
-      (effects (font (size 1.27 1.27)) hide)
-    )
-    (property "Value" "GND" (at 189.23 81.28 0)
-      (effects (font (size 1.27 1.27)))
-    )
-    (property "Footprint" "" (at 189.23 76.2 0)
-      (effects (font (size 1.27 1.27)) hide)
-    )
-    (property "Datasheet" "" (at 189.23 76.2 0)
+  (symbol (lib_id "power:GND") (at 123.19 77.47 0) (unit 1)
+    (in_bom yes) (on_board yes) (dnp no) (fields_autoplaced)
+    (property "Reference" "#PWR055" (at 123.19 83.82 0)
+      (effects (font (size 1.27 1.27)) hide)
+    )
+    (property "Value" "GND" (at 123.19 82.55 0)
+      (effects (font (size 1.27 1.27)))
+    )
+    (property "Footprint" "" (at 123.19 77.47 0)
+      (effects (font (size 1.27 1.27)) hide)
+    )
+    (property "Datasheet" "" (at 123.19 77.47 0)
       (effects (font (size 1.27 1.27)) hide)
     )
@@
     )
   )
-  (symbol (lib_id "Device:C_Small") (at 189.23 72.39 0) (unit 1)
-    (in_bom yes) (on_board yes) (dnp no) (fields_autoplaced)
-    (property "Reference" "C6" (at 191.77 71.1263 0)
-      (effects (font (size 1.27 1.27)) (justify left))
-    )
-    (property "Value" "330pF" (at 191.77 73.6663 0)
-      (effects (font (size 1.27 1.27)) (justify left))
-    )
-    (property "Footprint" "Capacitor_SMD:C_0805_2012Metric" (at 189.23 72.39 0)
-      (effects (font (size 1.27 1.27)) hide)
-    )
-    (property "Datasheet" "~" (at 189.23 72.39 0)
+  (symbol (lib_id "Device:C_Small") (at 123.19 72.39 0) (unit 1)
+    (in_bom yes) (on_board yes) (dnp no) (fields_autoplaced)
+    (property "Reference" "C6" (at 125.73 71.1263 0)
+      (effects (font (size 1.27 1.27)) (justify left))
+    )
+    (property "Value" "330pF" (at 125.73 73.6663 0)
+      (effects (font (size 1.27 1.27)) (justify left))
+    )
+    (property "Footprint" "Capacitor_SMD:C_0805_2012Metric" (at 123.19 72.39 0)
+      (effects (font (size 1.27 1.27)) hide)
+    )
+    (property "Datasheet" "~" (at 123.19 72.39 0)
       (effects (font (size 1.27 1.27)) hide)
     )
@@
         (path "/5cdf3b4f-d143-42e3-ac6f-eec5265de1fa/f403fb1f-6c3a-4b91-96f2-7610e89c4ca7"
           (reference "C7") (unit 1)
-        )
-      )
-    )
-  )
-  (symbol (lib_id "power:GND") (at 201.93 76.2 0) (unit 1)
-    (in_bom yes) (on_board yes) (dnp no) (fields_autoplaced)
-    (property "Reference" "#PWR056" (at 201.93 82.55 0)
-      (effects (font (size 1.27 1.27)) hide)
-    )
-    (property "Value" "GND" (at 201.93 81.28 0)
-      (effects (font (size 1.27 1.27)))
-    )
-    (property "Footprint" "" (at 201.93 76.2 0)
-      (effects (font (size 1.27 1.27)) hide)
-    )
-    (property "Datasheet" "" (at 201.93 76.2 0)
-      (effects (font (size 1.27 1.27)) hide)
-    )
-    (pin "1")
-    (instances
-      (project "ESPHome AIO"
-        (path "/5cdf3b4f-d143-42e3-ac6f-eec5265de1fa/f403fb1f-6c3a-4b91-96f2-7610e89c4ca7"
-          (reference "#PWR056") (unit 1)
         )
       )
@@
     )
   )
-  (symbol (lib_id "Device:C_Small") (at 201.93 72.39 0) (unit 1)
-    (in_bom yes) (on_board yes) (dnp no) (fields_autoplaced)
-    (property "Reference" "C8" (at 204.47 71.1263 0)
-      (effects (font (size 1.27 1.27)) (justify left))
-    )
-    (property "Value" "330pF" (at 204.47 73.6663 0)
-      (effects (font (size 1.27 1.27)) (justify left))
-    )
-    (property "Footprint" "Capacitor_SMD:C_0805_2012Metric" (at 201.93 72.39 0)
-      (effects (font (size 1.27 1.27)) hide)
-    )
-    (property "Datasheet" "~" (at 201.93 72.39 0)
-      (effects (font (size 1.27 1.27)) hide)
-    )
+  (symbol (lib_id "Device:C_Small") (at 134.62 72.39 0) (unit 1)
+    (in_bom yes) (on_board yes) (dnp no) (fields_autoplaced)
+    (property "Reference" "C8" (at 137.16 71.1263 0)
+      (effects (font (size 1.27 1.27)) (justify left))
+    )
+    (property "Value" "330pF" (at 137.16 73.6663 0)
+      (effects (font (size 1.27 1.27)) (justify left))
+    )
+    (property "Footprint" "Capacitor_SMD:C_0805_2012Metric" (at 134.62 72.39 0)
+      (effects (font (size 1.27 1.27)) hide)
+    )
+    (property "Datasheet" "~" (at 134.62 72.39 0)
+      (effects (font (size 1.27 1.27)) hide)
+    )
