File: KiCad Schematics and pcb/USB.kicad_sch (KiCad schematic)
At the start: 16 parts, among them IC4 TPS25730DREFR, J7 USB_C_Receptacle_USB2.0_16P, U1 TVS2200DRV

Commit message: V0.2 maybe
Parts:
- added R27, R33: 10K, Resistor_SMD:R_0805_2012Metric, symbol Device:R
- added R35: 110K, Resistor_SMD:R_0805_2012Metric, symbol Device:R
- added R36, R38: 1K, Resistor_SMD:R_0805_2012Metric, symbol Device:R
- added R37: 110k, Resistor_SMD:R_0805_2012Metric, symbol Device:R
- R14: value 10k -> 10K
- R16: value 6.8k -> 11K
Connections:
- net GND: now also R33.2, R36.2, R38.2; no longer IC4.2 (ADCIN1), IC4.5 (ADCIN3)
- net LDO_3V3: now also R27.1, R35.1, R37.1; no longer IC4.7 (ADCIN4)
- net ADC2: now reaches IC4.3 (ADCIN2), R15.2, R16.1
- new net ADC1: IC4.2 (ADCIN1), R37.2, R38.1
- new net ADC3: IC4.5 (ADCIN3), R35.2, R36.1
- new net ADC4: IC4.7 (ADCIN4), R27.2, R33.1
Other:
- note added: "USB Power Delivery controller set to negotiate for 12V 3A"
- note removed: "USB Power Delivery controller set to negotiate for 12V 5A"
- moved on the sheet: C3, R15, R16

Commit message: V0.2 wip
Parts:
- R16: value 11K -> 24K
Changed lines of the file:
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@@
   (junction (at 210.82 16.51) (diameter 0) (color 0 0 0 0)
+  )
+  (junction (at 53.34 16.51) (diameter 0) (color 0 0 0 0)
   )
   (junction (at 227.33 52.07) (diameter 0) (color 0 0 0 0)
@@
     (stroke (width 0) (type default))
   )
+  (wire (pts (xy 196.85 16.51) (xy 196.85 22.86))
+    (stroke (width 0) (type default))
+  )
+  (wire (pts (xy 106.68 76.2) (xy 109.22 76.2))
+    (stroke (width 0) (type default))
+  )
+  (wire (pts (xy 228.6 58.42) (xy 227.33 58.42))
+    (stroke (width 0) (type default))
+  )
+  (wire (pts (xy 53.34 45.72) (xy 60.96 45.72))
+    (stroke (width 0) (type default))
+  )
+  (wire (pts (xy 256.54 30.48) (xy 256.54 31.75))
+    (stroke (width 0) (type default))
+  )
+  (wire (pts (xy 39.37 101.6) (xy 63.5 101.6))
+    (stroke (width 0) (type default))
+  )
+  (wire (pts (xy 106.68 55.88) (xy 116.205 55.88))
+    (stroke (width 0) (type default))
+  )
+  (wire (pts (xy 248.92 115.57) (xy 254 115.57))
+    (stroke (width 0) (type default))
+  )
+  (wire (pts (xy 163.195 25.4) (xy 163.195 29.21))
+    (stroke (width 0) (type default))
+  )
+  (wire (pts (xy 210.82 40.64) (xy 205.74 40.64))
+    (stroke (width 0) (type default))
+  )
+  (wire (pts (xy 145.415 96.52) (xy 145.415 98.425))
+    (stroke (width 0) (type default))
+  )
+  (wire (pts (xy 146.685 24.765) (xy 146.685 28.575))
+    (stroke (width 0) (type default))
+  )
   (wire (pts (xy 53.34 16.51) (xy 58.42 16.51))
     (stroke (width 0) (type default))
   )
-  (wire (pts (xy 196.85 16.51) (xy 196.85 22.86))
-    (stroke (width 0) (type default))
-  )
-  (wire (pts (xy 106.68 76.2) (xy 109.22 76.2))
-    (stroke (width 0) (type default))
-  )
-  (wire (pts (xy 228.6 58.42) (xy 227.33 58.42))
-    (stroke (width 0) (type default))
-  )
-  (wire (pts (xy 53.34 45.72) (xy 60.96 45.72))
-    (stroke (width 0) (type default))
-  )
-  (wire (pts (xy 256.54 30.48) (xy 256.54 31.75))
-    (stroke (width 0) (type default))
-  )
-  (wire (pts (xy 39.37 101.6) (xy 63.5 101.6))
-    (stroke (width 0) (type default))
-  )
-  (wire (pts (xy 106.68 55.88) (xy 116.205 55.88))
-    (stroke (width 0) (type default))
-  )
-  (wire (pts (xy 248.92 115.57) (xy 254 115.57))
-    (stroke (width 0) (type default))
-  )
-  (wire (pts (xy 163.195 25.4) (xy 163.195 29.21))
-    (stroke (width 0) (type default))
-  )
-  (wire (pts (xy 210.82 40.64) (xy 205.74 40.64))
-    (stroke (width 0) (type default))
-  )
-  (wire (pts (xy 145.415 96.52) (xy 145.415 98.425))
-    (stroke (width 0) (type default))
-  )
-  (wire (pts (xy 146.685 24.765) (xy 146.685 28.575))
-    (stroke (width 0) (type default))
-  )
   (wire (pts (xy 227.33 53.34) (xy 227.33 52.07))
     (stroke (width 0) (type default))
@@
   )
   (wire (pts (xy 106.68 78.74) (xy 109.22 78.74))
+    (stroke (width 0) (type default))
+  )
+  (wire (pts (xy 50.8 16.51) (xy 53.34 16.51))
     (stroke (width 0) (type default))
   )
@@
   )
   (hierarchical_label "I2C_SDA" (shape input) (at 59.69 93.98 180) (fields_autoplaced)
+    (effects (font (size 1.27 1.27)) (justify right))
+  )
+  (hierarchical_label "VBUS" (shape input) (at 50.8 16.51 180) (fields_autoplaced)
     (effects (font (size 1.27 1.27)) (justify right))
   )
@@
       (effects (font (size 1.27 1.27)) (justify left))
     )
-    (property "Value" "11K" (at 165.1 45.72 0)
-      (effects (font (size 1.27 1.27)) (justify left))
-    )
+    (property "Value" "24K" (at 165.1 45.72 0)
+      (effects (font (size 1.27 1.27)) (justify left))
+    )

Commit message: 0.2
Parts:
- added D9: ESDALD05UE2X, SOT95P240X115-3N, symbol ComponentSearch:ESDALD05UE2X
Connections:
- net D+: now also D9.1 (I/O1)
- net D-: now also D9.2 (I/O2)
- net GND: now also D9.3 (GND)
