File: KiCad Schematics and pcb/ESPHome AIO.kicad_pcb (KiCad board)
At the start: 2 copper layers, 103 parts, among them IC1 ESP32-S3-WROOM-1-N8, IC2 EMC2101-ACZL-TR, IC3 TPS25730DREFR, IC4 LD1085D2T33R, IC5 BD50FC0FP-E2, J1 Conn_01x05, J10 Conn_01x04, J11 Conn_01x04, J12 Conn_01x04, J13 Screw_Terminal_01x03, J2 Conn_02x12_Top_Bottom, J3 Conn_01x04, J4 Conn_01x02_Pin, J4 Conn_01x04, J5 Screw_Terminal_01x06, J6 USB_C_Receptacle_USB2.0_16P, J7 Screw_Terminal_01x02, J8 694106301002, J9 Conn_01x04, M1 Fan_4pin, M2 Fan_4pin, M3 Fan_4pin, M4 Fan_4pin, Q1 DMN4035L-7, Q10 DMN4035L-7, Q11 DMN4035L-7, Q12 DMN4035L-7, Q13 2N7002NXAKR, Q2 DMN4035L-7, Q3 DMN4035L-7, Q4 DMN4035L-7, Q5 DMN4035L-7, Q6 DMN4035L-7, Q7 DMN4035L-7, Q8 DMN4035L-7, Q9 DMN4035L-7, SW1 SW_DPDT_x2, SW2 SW_DPDT_x2, SW3 SW_DPDT_x2, SW4 SW_DPDT_x2, SW5 SW_DPDT_x2, SW6 SW_DPDT_x2, SW7 SW_DPDT_x2, SW8 SW_DPDT_x2, U1 TVS2200DRV

Commit message: start pcb
Parts:
- removed D4, D5: LED, LED_SMD:LED_0805_2012Metric
- removed the Q10 at (142.4, 154.8)
- removed Q11: DMN4035L-7, ComponentSearch:SOT96P240X110-3N
- removed the R19 at (137.8, 154.0)
- removed the R20 at (137.8, 157.0)
- removed the R21 at (137.8, 159.9)
- removed the R22 at (178.4, 94.2)
- removed R23: 10K, Resistor_SMD:R_0805_2012Metric
- removed R24: 33K, Resistor_SMD:R_0805_2012Metric
- added IC1: TB67H451FNG,EL, ComponentSearch:SOIC127P600X170-9N, F.Cu at (138.9, 101.3)
- added M1: Motor_DC, Connector_Phoenix_MSTB:PhoenixContact_MSTBA_2,5_2-G-5,08_1x02_P5.08mm_Horizontal, F.Cu at (139.3, 87.0)
- added R1: 10KOhm, Resistor_SMD:R_0805_2012Metric, F.Cu at (124.5, 48.7)
- added R2: 10KOhm, Resistor_SMD:R_0805_2012Metric, F.Cu at (124.5, 51.6)
- added SW1: SW_Push, Button_Switch_THT:SW_PUSH_6mm_H7.3mm, F.Cu at (128.9, 43.1)
- added SW2: SW_Push, Button_Switch_THT:SW_PUSH_6mm_H7.3mm, F.Cu at (128.9, 51.7)
- J1: renamed from J2; footprint Connector_PinHeader_2.54mm:PinHeader_1x04_P2.54mm_Vertical -> Connector_PinHeader_2.54mm:PinHeader_2x12_P2.54mm_Vertical
- J11: renamed from J10; footprint Connector_Phoenix_MSTB:PhoenixContact_MSTBA_2,5_2-G-5,08_1x02_P5.08mm_Horizontal -> Connector_PinHeader_2.54mm:PinHeader_1x04_P2.54mm_Vertical
- J4: footprint Connector_PinHeader_2.54mm:PinHeader_1x04_P2.54mm_Vertical -> Connector_JST:JST_XH_B2B-XH-A_1x02_P2.50mm_Vertical
- J6: renamed from J13; footprint Connector_PinHeader_2.54mm:PinHeader_2x12_P2.54mm_Vertical -> Connector_Phoenix_MSTB:PhoenixContact_MSTBA_2,5_3-G-5,08_1x03_P5.08mm_Horizontal
- J8: renamed from J7; footprint ComponentSearch:694106301002_1 -> Connector_Phoenix_MSTB:PhoenixContact_MSTBA_2,5_2-G-5,08_1x02_P5.08mm_Horizontal
- J9: renamed from J8; footprint Connector_JST:JST_XH_B2B-XH-A_1x02_P2.50mm_Vertical -> ComponentSearch:694106301002_1
- U1: moved to F.Cu
- moved IC2 203.0 mm to (267.9, 88.5), turned to -90 degrees
- moved Q9 202.3 mm to (151.1, -40.0)
- moved R17 202.3 mm to (146.5, -40.9)
- moved R18 202.3 mm to (146.5, -37.9)
- moved D2 201.8 mm to (151.2, -35.6)
- moved R19 201.6 mm to (146.3, -34.2)
- moved Q10 185.1 mm to (150.9, -10.8)
- moved D3 185.1 mm to (150.8, -7.00)
- moved R20 185.1 mm to (146.3, -11.6)
- moved R21 185.1 mm to (146.3, -8.65)
- moved R22 185.1 mm to (146.3, -5.70)
- moved J6 182.8 mm to (270.1, 152.8), turned to 90 degrees
- moved Q8 167.4 mm to (263.9, 151.1)
- moved R12 167.4 mm to (263.7, 144.4)
- moved R13 167.4 mm to (263.7, 147.4)
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- renumbered IC1 to IC2, IC2 to IC3, IC3 to IC4, IC4 to IC5, IC5 to IC6, J9 to J10, J11 to J12, J12 to J13, J3 to J2, J1 to J3, J6 to J7, M1 to M2, M2 to M3, M3 to M4, M4 to M5, Q9 to Q10, Q12 to Q13, Q13 to Q8, Q8 to Q9, R8 to R10, R9 to R11, R28 to R12, R29 to R13, R10 to R14, R11 to R15, R12 to R16, R13 to R17, R14 to R18, R15 to R19, R16 to R20, R17 to R21, R18 to R22, R25 to R29, R1 to R3, R26 to R30, R27 to R31, R2 to R4, R3 to R5, R4 to R6, R5 to R7, R6 to R8, R7 to R9, SW8 to SW10, SW1 to SW3, SW2 to SW4, SW3 to SW5, SW4 to SW6, SW5 to SW7, SW6 to SW8, SW7 to SW9, TP2 to TP1, TP1 to TP2
Connections:
- net FAN renamed /Fan Headers/FAN
- net FAULT_IN renamed Net-(IC4-~{FAULT_IN})
- net MOS renamed /Fan Headers/MOS
- net Net-(C5-Pad1) renamed /USB/VBUS
- net Net-(D1-A) renamed /USB/USB_POWER
- net PLUG_EVENT renamed /USB/PLUG_EVENT
- net SINK_EN renamed /USB/SINK_EN
- net TACH renamed /Fan Headers/TACH
- net USB_PD_POWER renamed /USB_PD_POWER
- IC2 pad 10: /HPin15 -> /H.R5
- IC2 pad 11: /HPin16 -> /Motor_in1
- IC2 pad 12: /HPin17 -> /Motor_in2
- IC2 pad 26: /HPin9 -> unconnected-(IC2-IO45-Pad26)
- IC2 pad 27: /HPin8 -> /ARGB
- IC2 pad 28: unconnected-(IC1-IO35-Pad28) -> /Button2
- IC2 pad 29: unconnected-(IC1-IO36-Pad29) -> /Button1
- IC2 pad 30: unconnected-(IC1-IO37-Pad30) -> /H.L8
- IC2 pad 31: /HPin7 -> /H.L7
- IC2 pad 32: /HPin6 -> /H.L6
- IC2 pad 33: /HPin5 -> /H.L5
- IC2 pad 34: /HPin4 -> /H.L4
- IC2 pad 35: /HPin3 -> /H.L3
- IC2 pad 38: /HPin2 -> /H.L2
- IC2 pad 39: /HPin1 -> /H.L1
- IC2 pad 4: /HPin0 -> /H.L0
- IC2 pad 5: /HPin10 -> /H.R0
- IC2 pad 6: /HPin11 -> /H.R1
- IC2 pad 7: /HPin12 -> /H.R2
- IC2 pad 8: /HPin13 -> /H.R3
- IC2 pad 9: /HPin14 -> /H.R4
- IC4 pad 10: DBG_ACC -> unconnected-(IC4-DBG_ACC-Pad10)
- IC4 pad 13: PLUG_FLIP -> unconnected-(IC4-PLUG_FLIP-Pad13)
- IC4 pad 6: CAP_MIS -> /USB/CAP_MIS
- IC4 pad 8: I2C/SMdata -> /I2C/SMdata
- IC4 pad 9: I2C/SMclk -> /I2C/SMclk
- J1 pad 1: GND -> +3.3V
- J1 pad 2: +3.3V -> GND
- J1 pad 3: /HPin0 -> +5V
- J1 pad 4: /HPin1 -> /H.L0
- Q8 pad 2: /HPin9 -> /ARGB
- R12 pad 2: /HPin9 -> /ARGB
- R17 pad 2: CAO_MIS -> /USB/CAP_MIS
- R18 pad 1: CAO_MIS -> /USB/CAP_MIS
- SW6 pad 1: Net-(J10-Pin_3) (its old number) -> Net-(J11-Pin_3)
- SW6 pad 3: Net-(J10-Pin_4) (its old number) -> Net-(J11-Pin_4)
- SW6 pad 4: Net-(J10-Pin_4) (its old number) -> Net-(J11-Pin_4)
- SW6 pad 6: Net-(J10-Pin_3) (its old number) -> Net-(J11-Pin_3)
Routing:
- net /USB_D-: track 0.00 -> 45.3 mm, vias 0 -> 1
- net /USB_D+: track 0.00 -> 43.0 mm, vias 0 -> 3
- net GND: track 0.00 -> 18.4 mm, vias 0 -> 14
- net LDO_3V3: track 0.00 -> 13.0 mm, vias 0 -> 3
- net Net-(IC4-CC2): track 0.00 -> 10.2 mm
- net Net-(IC4-CC1): track 0.00 -> 9.91 mm, vias 0 -> 2
- net Net-(IC4-ADCIN2): track 0.00 -> 6.34 mm
- net Net-(IC4-DRAIN_PAD): track 0.00 -> 4.88 mm, vias 0 -> 3
- net /I2C/SMclk: track 0.00 -> 4.50 mm
- net +5V: track 0.00 -> 4.38 mm
- net /I2C/SMdata: track 0.00 -> 4.37 mm
- net Net-(IC4-~{FAULT_IN}): track 0.00 -> 2.45 mm
- net /USB/VBUS: vias 0 -> 29
- net +3.3V: vias 0 -> 5
- added copper zone on F.Cu, net /USB/USB_POWER
- added copper zone on B.Cu, net /USB/VBUS
- added copper zone on F.Cu, net /USB/VBUS
- added copper zone on F.Cu, net /USB_PD_POWER
- added copper zone on F.Cu, net 5V-24V
- added copper zone on F.Cu, net GND
- added copper zone on B.Cu, net Net-(IC4-DRAIN_PAD)
Other:
- board outline added: 100 x 100 mm
- copper layers 2 -> 4

Commit message: done for the day
Parts:
- removed J12: Conn_01x04, Connector_PinHeader_2.54mm:PinHeader_1x04_P2.54mm_Vertical
- removed the J3 at (20.4, 62.2)
- removed the J4 at (25.0, 62.2)
- removed the J9 at (29.6, 62.2)
- removed SW7, SW9: SW_DPDT_x2, Button_Switch_THT:SW_CuK_JS202011CQN_DPDT_Straight
- removed TP3: CC2, TestPoint:TestPoint_Loop_D2.60mm_Drill1.4mm_Beaded
- removed TP4: CC1, TestPoint:TestPoint_Loop_D2.60mm_Drill1.4mm_Beaded
- J1: value Conn_02x12_Top_Bottom -> Conn_02x12_Odd_Even
- moved J1 235.9 mm to (255.8, 84.9), turned to -90 degrees
- moved J3 212.6 mm to (228.7, 23.1), turned to 90 degrees
- moved J2 181.3 mm to (214.8, 78.8)
- moved R7 178.9 mm to (207.5, 97.8)
- moved R10 177.9 mm to (202.6, 97.8)
- moved Q3 177.6 mm to (207.5, 101.0), turned to -90 degrees
- moved Q6 174.1 mm to (202.5, 101.0), turned to -90 degrees
- moved R8 170.7 mm to (197.3, 97.8)
- moved Q4 170.7 mm to (197.3, 101.0), turned to -90 degrees
- moved R11 170.0 mm to (192.4, 97.8)
- moved Q7 167.6 mm to (192.3, 101.0), turned to -90 degrees
- moved Q5 164.7 mm to (187.2, 101.0), turned to -90 degrees
- moved R9 162.9 mm to (187.2, 97.6)
- moved SW10 149.9 mm to (176.1, 87.1), turned to 90 degrees
- moved SW8 149.4 mm to (176.1, 77.2), turned to 90 degrees
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Connections:
- IC2 pad 15: /R -> /WW
- IC2 pad 16: /G -> /CW
- IC2 pad 18: /CW -> /G
- IC2 pad 19: /WW -> /R
- J1 pad 10: /H.L6 -> /I2C/SMdata
- J1 pad 11: /H.L7 -> /H.L2
- J1 pad 12: /H.L8 -> /I2C/SMclk
- J1 pad 13: +3.3V -> /H.L3
- J1 pad 14: GND -> /H.R0
- J1 pad 15: +5V -> /H.L4
- J1 pad 16: GND -> /H.R1
- J1 pad 17: /I2C/SMdata -> /H.L5
- J1 pad 18: /I2C/SMclk -> /H.R2
- J1 pad 19: /H.R0 -> /H.L6
- J1 pad 2: GND -> +3.3V
- J1 pad 20: /H.R1 -> /H.R3
- J1 pad 21: /H.R2 -> /H.L7
- J1 pad 22: /H.R3 -> /H.R4
- J1 pad 23: /H.R4 -> /H.L8
- J1 pad 3: +5V -> GND
- J1 pad 4: /H.L0 -> GND
- J1 pad 5: /H.L1 -> +5V
- J1 pad 6: /H.L2 -> +5V
- J1 pad 7: /H.L3 -> /H.L0
- J1 pad 8: /H.L4 -> GND
- J1 pad 9: /H.L5 -> /H.L1
- M1 pad 1: Net-(IC1-OUT2) -> Net-(IC1-OUT1)
- M1 pad 2: Net-(IC1-OUT1) -> Net-(IC1-OUT2)
Routing:
- net 5V-24V: track 0.00 -> 71.4 mm
- net /Fan Headers/FAN: track 0.00 -> 35.8 mm
- net GND: track 18.4 -> 40.5 mm, vias 14 -> 25
- net Net-(J10-Pin_2): track 0.00 -> 15.0 mm
- net Net-(J10-Pin_3): track 0.00 -> 14.9 mm
- net Net-(J10-Pin_4): track 0.00 -> 12.8 mm
- net Net-(J10-Pin_1): track 0.00 -> 12.7 mm
- net +3.3V: track 0.00 -> 11.7 mm, vias 5 -> 6
- net Net-(IC3-DP): track 0.00 -> 10.1 mm
- net +5V: track 4.38 -> 12.7 mm
- net /I2C/SMclk: track 4.50 -> 12.2 mm
- net Net-(IC3-DN): track 0.00 -> 6.80 mm
- net Net-(IC1-OUT2): track 0.00 -> 6.56 mm
- net Net-(IC1-OUT1): track 0.00 -> 6.43 mm
- net /I2C/SMdata: track 4.37 -> 10.0 mm
- added copper zone on In1.Cu, net +3.3V
- added copper zone on In2.Cu, net GND
Other:
- outline, holes or cut-outs redrawn

Commit message: posible V0.1
Parts:
- removed D6: LED, LED_SMD:LED_0805_2012Metric
- removed Q13: DMN4035L-7, ComponentSearch:SOT96P240X110-3N
- removed R29: 11K, Resistor_SMD:R_0805_2012Metric
- removed R30: 10K, Resistor_SMD:R_0805_2012Metric
- removed R31: 33K, Resistor_SMD:R_0805_2012Metric
- added H1: MountingHole, MountingHole:MountingHole_4.3mm_M4, F.Cu at (184.9, 45.7)
- added H2: MountingHole_Pad, MountingHole:MountingHole_4.3mm_M4_Pad, F.Cu at (95.1, 46.1)
- added H3: MountingHole_Pad, MountingHole:MountingHole_4.3mm_M4_Pad, F.Cu at (95.3, 135.4)
- added H4: MountingHole, MountingHole:MountingHole_4.3mm_M4, F.Cu at (184.9, 135.7)
- added TP3: Power, TestPoint:TestPoint_Loop_D2.60mm_Drill1.4mm_Beaded, F.Cu at (146.3, 59.2)
- added TP4: 3.3V, TestPoint:TestPoint_Loop_D2.60mm_Drill1.4mm_Beaded, F.Cu at (112.1, 83.1)
- TP5: value VBUS -> 5V
- moved TP5 91.0 mm to (140.3, 108.1)
- moved C13 87.4 mm to (119.3, 84.0)
- moved M2 85.1 mm to (169.1, 127.1)
- moved IC1 82.5 mm to (173.9, 60.0)
- moved M1 82.2 mm to (175.9, 51.4)
- moved M4 80.1 mm to (176.4, 127.1)
- moved M3 80.1 mm to (169.1, 138.4)
- moved SW1 79.7 mm to (119.3, 102.5)
- moved C10 79.3 mm to (136.4, 74.2)
- moved J4 79.3 mm to (177.7, 114.5)
- moved J6 79.3 mm to (146.4, 129.8)
- moved JP1 79.3 mm to (145.1, 69.5)
- moved C3 79.3 mm to (102.0, 57.5)
- moved C5 79.3 mm to (112.7, 55.2)
- moved C7 79.3 mm to (112.7, 51.2)
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Connections:
- IC2 pad 11: /Motor_in1 -> /Motor_in2
- IC2 pad 12: /Motor_in2 -> /Motor_in1
- IC2 pad 15: /WW -> /TX
- IC2 pad 16: /CW -> /RX
- IC2 pad 17: /B -> /LD2410_I/O
- IC2 pad 18: /G -> /WW
- IC2 pad 19: /R -> /CW
- IC2 pad 20: /TX -> /B
- IC2 pad 21: /RX -> /G
- IC2 pad 22: /LD2410_I/O -> /R
- J1 pad 1: +3.3V -> +5V
- J1 pad 2: +3.3V -> +5V
- J1 pad 5: +5V -> +3.3V
- J1 pad 6: +5V -> +3.3V
- J2 pad 3: /TX0 -> /RX0
- J2 pad 4: /RX0 -> /TX0
- SW10 pad 2: I2C/SMdata -> /I2C/SMdata
- SW10 pad 5: I2C/SMclk -> /I2C/SMclk
- SW5 pad 2: I2C/SMdata -> /I2C/SMdata
- SW5 pad 5: I2C/SMclk -> /I2C/SMclk
- SW6 pad 2: I2C/SMdata -> /I2C/SMdata
- SW6 pad 5: I2C/SMclk -> /I2C/SMclk
- TP5 pad 1: /USB/VBUS -> +5V
Routing:
- net /I2C/SMdata: track 10.0 -> 216.9 mm, vias 0 -> 7
- net /I2C/SMclk: track 12.2 -> 210.6 mm, vias 0 -> 6
- net /WW: track 0.00 -> 82.2 mm
- net /CW: track 0.00 -> 79.1 mm
- net /R: track 0.00 -> 77.3 mm
- net /B: track 0.00 -> 76.1 mm
- net /G: track 0.00 -> 76.0 mm
- net /Button1: track 0.00 -> 58.8 mm
- net /Button2: track 0.00 -> 54.0 mm
- net 5V-24V: track 71.4 -> 123.0 mm, vias 0 -> 10
- net /Fan_pwm/dc: track 0.00 -> 49.9 mm, vias 0 -> 2
- net /H.R5: track 0.00 -> 46.3 mm, vias 0 -> 1
- net /TX0: track 0.00 -> 45.7 mm, vias 0 -> 1
- net /H.R4: track 0.00 -> 45.7 mm, vias 0 -> 1
- net /ARGB: track 0.00 -> 45.4 mm, vias 0 -> 2
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- added copper zone on B.Cu, net +3.3V
- added copper zone on F.Cu, net +3.3V
- added copper zone on B.Cu, net +5V
- added copper zone on F.Cu, net +5V
- added copper zone on B.Cu, net 5V-24V
- added copper zone on B.Cu, net GND
- removed copper zone on In1.Cu, net +3.3V
- removed copper zone on In2.Cu, net GND
Other:
- outline, holes or cut-outs redrawn
- copper layers 4 -> 2
- board text added: "+"
- board text added: "+3.3V"
- board text added: "+5V"
- board text added: "5-24V"
- board text added: "5V"
- board text added: "B"
- board text added: "CW"
- board text added: "D"
- board text added: "Fan Header"
- board text added: "G"
- board text added: "GND"
- board text added: "Main Power"
- board text added: "R"
- board text added: "SCL"
- board text added: "SDA"
- board text added: "Sink"
- board text added: "Switch-> GND->"
- board text added: "Switch-> SCL->"
- board text added: "WW"
- board text added: "cap_mis"
- board text added: "fan temp sensor"

Commit message: v0.1 prototype ordered
Parts:
- added D4: LED, LED_SMD:LED_0805_2012Metric, F.Cu at (145.4, 82.4)
- added D5: LED, LED_SMD:LED_0805_2012Metric, F.Cu at (126.2, 88.7)
- added G***: Barrel_Polarity, ComponentSearch:Barrel_Polarity, F.Cu at (145.7, 45.8)
- added IC7: BZX84-C12, ComponentSearch:SOT95P230X110-3N, F.Cu at (149.3, 81.9)
- added IC8: TPS259573DSGR, ComponentSearch:SON50P200X200X80-9N, F.Cu at (143.0, 86.9)
- added IC9: TPS259573DSGR, ComponentSearch:SON50P200X200X80-9N, F.Cu at (119.8, 87.1)
- added JP2: SolderJumper_2_Bridged, Jumper:SolderJumper-2_P1.3mm_Open_TrianglePad1.0x1.5mm, F.Cu at (137.1, 79.8)
- added JP3: Jumper_3_Bridged12, Connector_PinHeader_2.54mm:PinHeader_1x03_P2.54mm_Vertical, F.Cu at (153.0, 86.2)
- added R23: 10K, Resistor_SMD:R_0805_2012Metric, F.Cu at (139.4, 87.0)
- added R24: 36.5K, Resistor_SMD:R_0805_2012Metric, F.Cu at (139.4, 83.5)
- added R25: 2.32K, Resistor_SMD:R_0805_2012Metric, F.Cu at (153.1, 89.8)
- added R26: 2.2K, Resistor_SMD:R_0805_2012Metric, F.Cu at (142.6, 81.4)
- added R27: 1K, Resistor_SMD:R_0805_2012Metric, F.Cu at (142.6, 83.4)
- added R28: 487, Resistor_SMD:R_0805_2012Metric, F.Cu at (147.9, 89.8)
- added R29: 715, Resistor_SMD:R_0805_2012Metric, F.Cu at (123.6, 85.5)
- added R30: 20.5K, Resistor_SMD:R_0805_2012Metric, F.Cu at (116.3, 86.0)
- added R31: 10K, Resistor_SMD:R_0805_2012Metric, F.Cu at (116.3, 89.5)
- added R32: 680, Resistor_SMD:R_0805_2012Metric, F.Cu at (123.5, 88.5)
- C4: value 0.1uF -> 100nF
- C7, C9: value 0.01uF -> 10nF
- F1: footprint Fuse:Fuseholder_Clip-5x20mm_Bel_FC-203-22_Lateral_P17.80x5.00mm_D1.17mm_Horizontal -> Fuse:Fuseholder_Littelfuse_Nano2_154x
- J9: value 694106301002 -> XKB Connection DC-005-5A-3.0; footprint ComponentSearch:694106301002_1 -> Connector_BarrelJack:BarrelJack_Horizontal
- M1: value Motor_DC -> Screw_Terminal_01x02
- R1, R2, R3, R4: value 10KOhm -> 10K
- R5, R6: value 2KOhm -> 2K
- moved TP4 19.3 mm to (131.2, 85.7)
- moved J9 14.4 mm to (139.0, 55.0)
- moved TP1 12.0 mm to (160.2, 87.4)
- moved TP3 9.87 mm to (140.0, 66.8)
- moved F1 5.79 mm to (128.3, 62.3)
- moved TP2 4.79 mm to (158.2, 91.5)
- moved R1 3.80 mm to (116.3, 107.2)
- moved R2 3.80 mm to (116.3, 98.0)
- moved SW1 3.80 mm to (119.3, 106.2)
- moved SW2 3.80 mm to (119.3, 97.0)
- moved J3 2.60 mm to (152.1, 46.4)
- moved D7 0.55 mm to (145.6, 65.0)
Connections:
- C12 pad 1: +5V -> Net-(IC6-VO)
- C13 pad 1: +3.3V -> Net-(IC5-OUTPUT)
- IC5 pad 4: +3.3V -> Net-(IC5-OUTPUT)
- IC6 pad 3: +5V -> Net-(IC6-VO)
- JP1 pad 2: +5V -> Net-(IC7-K)
Routing:
- net Net-(IC7-K): track 0.00 -> 51.7 mm
- net Net-(IC5-OUTPUT): track 0.00 -> 30.7 mm, vias 0 -> 2
- net GND: track 59.1 -> 79.4 mm, vias 54 -> 53
- net (no net): track 0.00 -> 13.2 mm, vias 0 -> 2
- net +5V: track 47.3 -> 60.0 mm, vias 13 -> 9
- net /R: track 77.3 -> 85.0 mm
- net Net-(IC8-ILM): track 0.00 -> 7.58 mm
- net /WW: track 82.2 -> 88.4 mm
- net Net-(D5-K): track 0.00 -> 5.57 mm
- net 5V-24V: track 123.0 -> 117.5 mm, vias 10 -> 9
- net /G: track 76.0 -> 81.4 mm
- net Net-(D4-K): track 0.00 -> 4.95 mm, vias 0 -> 2
- net Net-(IC8-~{EN}/OVLO): track 0.00 -> 4.45 mm
- net /B: track 76.1 -> 80.4 mm
- net /CW: track 79.1 -> 83.3 mm
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- added copper zone on F.Cu, net Net-(IC6-VO)
- removed copper zone on B.Cu, net +3.3V
Other:
- board text added: "-"
- board text added: "1A Limit ^"
- board text added: "4A Limit ^"
- board text added: "<- 5V Fault"
- board text added: "ARGB"
- board text added: "Don't forget to double check the switches"
- board text added: "ESP32-S3"
- board text added: "Fan Headers"
- board text added: "GND-> Switch->"
- board text added: "General purpose buttons"
- board text added: "I/O"
- board text added: "I2C/SMBus Headers"
- board text added: "Leftover I/O"
- board text added: "Motor Driver"
- board text added: "RGBWW"
- board text added: "RX"
- board text added: "SCL-> Switch->"
- board text added: "Serial Header"
- board text added: "TX"
- board text added: "^ 3.3V Fault"
- board text removed: "Fan Header"
- board text removed: "Switch-> GND->"
- board text removed: "Switch-> SCL->"

Commit message: V0.2 maybe
Parts:
- removed Q10: DMN4035L-7, ComponentSearch:SOT96P240X110-3N
- added C14: 100nF, Capacitor_SMD:C_0805_2012Metric, F.Cu at (178.5, 66.5)
- added Q11: 2N7002NXAKR, ComponentSearch:SOT95P230X110-3N, F.Cu at (94.6, 67.3)
- added Q12: 2N7002NXAKR, ComponentSearch:SOT95P230X110-3N, F.Cu at (111.0, 74.8)
- added R27: 10K, Resistor_SMD:R_0805_2012Metric, F.Cu at (98.8, 67.8)
- added R33: 10K, Resistor_SMD:R_0805_2012Metric, F.Cu at (102.5, 67.8)
- added R34: 10K, Resistor_SMD:R_0805_2012Metric, F.Cu at (154.8, 114.7)
- added R35: 110K, Resistor_SMD:R_0805_2012Metric, F.Cu at (98.8, 65.3)
- added R36: 1K, Resistor_SMD:R_0805_2012Metric, F.Cu at (102.3, 65.3)
- added R37: 110k, Resistor_SMD:R_0805_2012Metric, F.Cu at (99.1, 55.6)
- added R38: 1K, Resistor_SMD:R_0805_2012Metric, F.Cu at (95.5, 55.6)
- added R39: 10K, Resistor_SMD:R_0805_2012Metric, F.Cu at (172.6, 64.6)
- added SW7: SW_Push, Button_Switch_THT:SW_PUSH_6mm_H7.3mm, F.Cu at (176.2, 63.9)
- Q9: value DMN4035L-7 -> 2N7002NXAKR; footprint ComponentSearch:SOT96P240X110-3N -> ComponentSearch:SOT95P230X110-3N
- R14: value 10k -> 10K
- R16: value 6.8k -> 11K
- moved Q9 41.7 mm to (129.8, 89.8)
- moved IC1 7.90 mm to (166.0, 60.0)
- moved D2 1.52 mm to (95.7, 60.1)
- moved R17 1.52 mm to (92.8, 60.1)
- moved R18 1.52 mm to (92.8, 63.6)
- moved R19 1.52 mm to (95.7, 63.8)
Connections:
- net Net-(IC4-ADCIN2) renamed /USB/ADC2
- D5 pad 2: Net-(D5-A) -> /Power/3.3V_FLT
- IC2 pad 3: +3.3V -> /EN
- IC4 pad 2: GND -> /USB/ADC1
- IC4 pad 5: GND -> /USB/ADC3
- IC4 pad 7: LDO_3V3 -> /USB/ADC4
- Q9 pad 1: Net-(Q9-G) -> /Power/3.3V_FLT
- Q9 pad 2: GND -> Net-(Q9-S)
- Q9 pad 3: Net-(Q9-D) -> Net-(IC8-~{EN}/OVLO)
- R18 pad 2: Net-(Q9-G) -> Net-(Q11-G)
- R19 pad 2: Net-(Q9-D) -> Net-(Q11-D)
- R23 pad 1: Net-(IC8-~{EN}/OVLO) -> Net-(Q9-S)
- R32 pad 2: Net-(D5-A) -> /Power/3.3V_FLT
Routing:
- net +3.3V: track 8.04 -> 41.5 mm, vias 2 -> 4
- net LDO_3V3: track 25.2 -> 49.4 mm, vias 3 -> 4
- net /EN: track 0.00 -> 17.2 mm
- net Net-(Q9-S): track 0.00 -> 16.1 mm, vias 0 -> 2
- net Net-(IC8-~{EN}/OVLO): track 4.45 -> 17.9 mm, vias 0 -> 2
- net (no net): track 13.2 -> 0.00 mm, vias 2 -> 0
- net /USB/ADC4: track 0.00 -> 12.7 mm
- net /USB/ADC1: track 0.00 -> 11.7 mm
- net GND: track 79.4 -> 89.0 mm, vias 53 -> 55
- net /USB/ADC3: track 0.00 -> 8.51 mm
- net 5V-24V: track 117.5 -> 109.2 mm
- net /USB/CAP_MIS: track 15.6 -> 23.4 mm
- net Net-(IC1-OUT1): track 6.71 -> 13.0 mm
- net /Power/3.3V_FLT: track 0.00 -> 5.03 mm
- net Net-(IC1-OUT2): track 6.68 -> 9.88 mm
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Other:
- board text added: "3.3V Fault ^"
- board text removed: "^ 3.3V Fault"
