File: KiCad Schematics and pcb/ESPHome AIO.kicad_pcb (KiCad board)
At the start: 2 copper layers, 100 x 100 mm, 122 parts, among them IC1 TB67H451FNG,EL, IC2 ESP32-S3-WROOM-1-N8, IC3 EMC2101-ACZL-TR, IC4 TPS25730DREFR, IC5 LD1085D2T33R, IC6 BD50FC0FP-E2, IC7 BZX84-C12, IC8 TPS259573DSGR, IC9 TPS259573DSGR, J1 Conn_02x12_Odd_Even, J10 Conn_01x04, J11 Conn_01x04, J13 Conn_01x04, J2 Conn_01x04, J3 Conn_01x05, J4 Conn_01x02_Pin, J5 Screw_Terminal_01x06, J6 Screw_Terminal_01x03, J7 USB_C_Receptacle_USB2.0_16P, J8 Screw_Terminal_01x02, J9 XKB Connection DC-005-5A-3.0, M1 Screw_Terminal_01x02, M2 Fan_4pin, M3 Fan_4pin, M4 Fan_4pin, M5 Fan_4pin, Q1 DMN4035L-7, Q11 2N7002NXAKR, Q12 2N7002NXAKR, Q2 DMN4035L-7, Q3 DMN4035L-7, Q4 DMN4035L-7, Q5 DMN4035L-7, Q6 DMN4035L-7, Q7 DMN4035L-7, Q8 2N7002NXAKR, Q9 2N7002NXAKR, SW1 SW_Push, SW10 SW_DPDT_x2, SW2 SW_Push, SW3 SW_DPDT_x2, SW4 SW_DPDT_x2, SW5 SW_DPDT_x2, SW6 SW_DPDT_x2, SW7 SW_Push, SW8 SW_DPDT_x2, U1 TVS2200DRV

Commit message: 0.2
Parts:
- added D8: LED, LED_SMD:LED_0805_2012Metric, F.Cu at (138.2, 62.6)
- added D9: ESDALD05UE2X, ComponentSearch:SOT95P240X115-3N, F.Cu at (151.7, 55.2)
- added JP4: Jumper_2_Open, Connector_PinHeader_2.54mm:PinHeader_1x02_P2.54mm_Vertical, F.Cu at (142.4, 116.0)
- added R40: 10K, Resistor_SMD:R_0805_2012Metric, F.Cu at (142.4, 61.7)
- J9: footprint ComponentSearch:694106301002_1 -> Connector_BarrelJack:BarrelJack_Horizontal
- Q1, Q2, Q3, Q4, Q5, Q6, Q7: value DMN4035L-7 -> RQ3E080BNTB; footprint ComponentSearch:SOT96P240X110-3N -> ComponentSearch:RQ3E080BNTB
- R17, R20: value 11K -> 10K
- R19, R22: value 33K -> 10K
- SW10, SW3, SW4, SW5, SW6, SW8: footprint Button_Switch_THT:SW_CuK_JS202011CQN_DPDT_Straight -> ComponentSearch:SW_CK_JS202011CQN_DPDT_Straight
- moved J9 14.2 mm to (139.0, 54.8)
- moved Q6 10.5 mm to (115.4, 122.2), turned to 90 degrees
- moved Q5 10.2 mm to (120.8, 122.2), turned to 90 degrees
- moved Q7 5.77 mm to (110.0, 122.2), turned to 90 degrees
- moved Q4 5.55 mm to (126.2, 122.2), turned to 90 degrees
- moved Q2 5.44 mm to (162.2, 124.6), turned to 180 degrees
- moved Q1 4.67 mm to (162.2, 119.2), turned to 180 degrees
- moved Q3 0.90 mm to (131.6, 122.2), turned to 90 degrees
- moved R10 0.20 mm to (126.0, 118.3)
- moved R8 0.20 mm to (120.8, 118.3)
- moved R11 0.20 mm to (115.8, 118.3)
- moved R7 0.20 mm to (130.9, 118.3)
Connections:
- C10 pad 1: /USB/VBUS -> 5V-24V
- IC1 pad 2: /Motor_in1 -> /Motor_in2
- IC1 pad 3: /Motor_in2 -> /Motor_in1
- IC2 pad 11: /Motor_in2 -> /Motor_in1
- IC2 pad 12: /Motor_in1 -> /Motor_in2
- IC5 pad 3: /USB/VBUS -> 5V-24V
- Q1 pad 1: /Fan Headers/FAN -> GND
- Q1 pad 3: /Fan Headers/MOS -> GND
- Q2 pad 1: /Fan_pwm/dc -> GND
- Q2 pad 3: /Fan Headers/MOS -> GND
- Q3 pad 1: /R -> GND
- Q3 pad 3: Net-(J5-Pin_5) -> GND
- Q4 pad 1: /B -> GND
- Q4 pad 3: Net-(J5-Pin_3) -> GND
- Q5 pad 1: /WW -> GND
- Q5 pad 3: Net-(J5-Pin_1) -> GND
- Q6 pad 1: /G -> GND
- Q6 pad 3: Net-(J5-Pin_4) -> GND
- Q7 pad 1: /CW -> GND
- Q7 pad 3: Net-(J5-Pin_2) -> GND
Routing:
- net /USB/VBUS: track 30.9 -> 0.00 mm, vias 25 -> 24
- net /ARGB: track 45.1 -> 54.3 mm
- net Net-(IC5-OUTPUT): track 30.7 -> 37.7 mm
- net 5V-24V: track 109.2 -> 113.2 mm
- net /Fan Headers/MOS: track 39.0 -> 42.5 mm
- net GND: track 93.0 -> 89.6 mm, vias 55 -> 63
- net Net-(D8-K): track 0.00 -> 3.32 mm
- net /USB_D-: track 83.1 -> 84.7 mm, vias 2 -> 4
- net /R: track 85.0 -> 86.6 mm
- net /USB_D+: track 80.3 -> 81.6 mm, vias 4 -> 6
- net +5V: track 60.1 -> 58.9 mm
- net /G: track 81.4 -> 82.5 mm
- net /B: track 80.4 -> 81.4 mm
- net Net-(J5-Pin_1): track 7.12 -> 8.01 mm
- net /CW: track 83.3 -> 84.2 mm
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Other:
- board text added: "Boot"
- board text added: "Power"
