File: KiCad Schematics and pcb/_autosave-ESPHome AIO.kicad_pcb (KiCad board)
At the start: 2 copper layers, 100 x 100 mm, 122 parts, among them IC1 TB67H451FNG,EL, IC2 ESP32-S3-WROOM-1-N8, IC3 EMC2101-ACZL-TR, IC4 TPS25730DREFR, IC5 LD1085D2T33R, IC6 BD50FC0FP-E2, IC7 BZX84-C12, IC8 TPS259573DSGR, IC9 TPS259573DSGR, J1 Conn_02x12_Odd_Even, J10 Conn_01x04, J11 Conn_01x04, J13 Conn_01x04, J2 Conn_01x04, J3 Conn_01x05, J4 Conn_01x02_Pin, J5 Screw_Terminal_01x06, J6 Screw_Terminal_01x03, J7 USB_C_Receptacle_USB2.0_16P, J8 Screw_Terminal_01x02, J9 XKB Connection DC-005-5A-3.0, M1 Screw_Terminal_01x02, M2 Fan_4pin, M3 Fan_4pin, M4 Fan_4pin, M5 Fan_4pin, Q1 DMN4035L-7, Q11 2N7002NXAKR, Q12 2N7002NXAKR, Q2 DMN4035L-7, Q3 DMN4035L-7, Q4 DMN4035L-7, Q5 DMN4035L-7, Q6 DMN4035L-7, Q7 DMN4035L-7, Q8 2N7002NXAKR, Q9 2N7002NXAKR, SW1 SW_Push, SW10 SW_DPDT_x2, SW2 SW_Push, SW3 SW_DPDT_x2, SW4 SW_DPDT_x2, SW5 SW_DPDT_x2, SW6 SW_DPDT_x2, SW7 SW_Push, SW8 SW_DPDT_x2, U1 TVS2200DRV

Commit message: V0.2 wip
Connections:
- IC1 pad 2: /Motor_in1 -> /Motor_in2
- IC1 pad 3: /Motor_in2 -> /Motor_in1
- IC2 pad 11: /Motor_in2 -> /Motor_in1
- IC2 pad 12: /Motor_in1 -> /Motor_in2
Changed lines of the file:
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@@
       (net 1 "GND") (pinfunction "GND") (pintype "power_in"))
     (pad "2" smd rect (at -2.475 -0.635 180) (size 0.65 2) (layers "F.Cu" "F.Paste" "F.Mask")
-      (net 16 "/Motor_in1") (pinfunction "IN2") (pintype "input"))
+      (net 28 "/Motor_in2") (pinfunction "IN2") (pintype "input"))
     (pad "3" smd rect (at -2.475 0.635 180) (size 0.65 2) (layers "F.Cu" "F.Paste" "F.Mask")
-      (net 28 "/Motor_in2") (pinfunction "IN1") (pintype "input"))
+      (net 16 "/Motor_in1") (pinfunction "IN1") (pintype "input"))
     (pad "4" smd rect (at -2.475 1.905 180) (size 0.65 2) (layers "F.Cu" "F.Paste" "F.Mask")
       (net 5 "+3.3V") (pinfunction "VREF") (pintype "input"))
@@
       (net 15 "/H.R5") (pinfunction "IO17") (pintype "bidirectional"))
     (pad "11" smd rect (at -8.75 7.44) (size 0.9 1.5) (layers "F.Cu" "F.Paste" "F.Mask")
-      (net 28 "/Motor_in2") (pinfunction "IO18") (pintype "bidirectional"))
+      (net 16 "/Motor_in1") (pinfunction "IO18") (pintype "bidirectional"))
     (pad "12" smd rect (at -8.75 8.71) (size 0.9 1.5) (layers "F.Cu" "F.Paste" "F.Mask")
-      (net 16 "/Motor_in1") (pinfunction "IO8") (pintype "bidirectional"))
+      (net 28 "/Motor_in2") (pinfunction "IO8") (pintype "bidirectional"))
     (pad "13" smd rect (at -8.75 9.98) (size 0.9 1.5) (layers "F.Cu" "F.Paste" "F.Mask")
       (net 17 "/USB_D-") (pinfunction "IO19") (pintype "bidirectional"))
@@
   (segment (start 152.6 106.78) (end 151.28 108.1) (width 0.3) (layer "B.Cu") (net 15))
   (segment (start 152.6 105.082943) (end 152.6 106.78) (width 0.3) (layer "B.Cu") (net 15))
-  (segment (start 165.405 64.145) (end 168.33 67.07) (width 0.5) (layer "F.Cu") (net 16))
-  (segment (start 168.33 67.07) (end 168.33 69.95) (width 0.5) (layer "F.Cu") (net 16))
-  (segment (start 165.405 62.475) (end 165.405 64.145) (width 0.5) (layer "F.Cu") (net 16))
+  (segment (start 169.6 67.07) (end 169.6 69.95) (width 0.5) (layer "F.Cu") (net 16))
+  (segment (start 166.675 64.145) (end 166.675 62.475) (width 0.5) (layer "F.Cu") (net 16))
+  (segment (start 166.675 64.145) (end 169.6 67.07) (width 0.5) (layer "F.Cu") (net 16))
   (segment (start 108.45 48.775) (end 108.4 48.725) (width 0.2) (layer "F.Cu") (net 17))
   (segment (start 108.45 48.775) (end 108.425001 48.799999) (width 0.2) (layer "F.Cu") (net 17))
@@
   (segment (start 162.5 92.360788) (end 162.5 81.9) (width 0.3) (layer "B.Cu") (net 27))
   (segment (start 153.275 100.5) (end 154.360788 100.5) (width 0.3) (layer "B.Cu") (net 27))
-  (segment (start 169.6 67.07) (end 169.6 69.95) (width 0.5) (layer "F.Cu") (net 28))
-  (segment (start 166.675 64.145) (end 166.675 62.475) (width 0.5) (layer "F.Cu") (net 28))
-  (segment (start 166.675 64.145) (end 169.6 67.07) (width 0.5) (layer "F.Cu") (net 28))
+  (segment (start 165.405 64.145) (end 168.33 67.07) (width 0.5) (layer "F.Cu") (net 28))
+  (segment (start 168.33 67.07) (end 168.33 69.95) (width 0.5) (layer "F.Cu") (net 28))
+  (segment (start 165.405 62.475) (end 165.405 64.145) (width 0.5) (layer "F.Cu") (net 28))
   (segment (start 153.35 98.25) (end 151.95 98.25) (width 0.3) (layer "F.Cu") (net 29))
   (segment (start 148.9 117.1) (end 149.5425 117.7425) (width 0.3) (layer "F.Cu") (net 29))
