File: KiCad Schematics and pcb/FanHeaders.kicad_sch (KiCad schematic)
At the start: 10 parts, among them IC2 EMC2101-ACZL-TR, J4 Conn_01x02_Pin, M1 Fan_4pin, M2 Fan_4pin, M3 Fan_4pin, M4 Fan_4pin, Q1 DMN4035L-7, Q2 DMN4035L-7

Commit message: start pcb
Parts:
- IC3: renamed from IC2; footprint SOP65P490X110-8N -> ComponentSearch:SOP65P490X110-8N
- J4: footprint Connector_PinHeader_2.54mm:PinHeader_1x04_P2.54mm_Vertical -> Connector_JST:JST_XH_B2B-XH-A_1x02_P2.50mm_Vertical
- Q1, Q2: footprint SOT96P240X110-3N -> ComponentSearch:SOT96P240X110-3N
- renumbered M1 to M2, M2 to M3, M3 to M4, M4 to M5, R3 to R5, R4 to R6

Commit message: v0.1
Other:
- note added: "Fan Connectors"
- note added: "Fan Controller"
- moved on the sheet: IC3, J4, M2, M3, M4, M5, Q1, Q2, R5, R6

Commit message: v0.1 prototype ordered
Parts:
- R5, R6: value 2KOhm -> 2K
Other:
- note added: "Only fan header M2 has the Tach connected. The fan controller will adjust pwm only depending on the speed of M2. So make sure to use M2 first. Also i suggest not mixing fans if you are using the power pin to adjust speed."
- note removed: "Only fan header M1 has the Tach connected. The fan controller will adjust pwm only depending on the speed of M1. So make sure to use M1 first"
Changed lines of the file:
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@@
     (effects (font (size 1.27 1.27)) (justify left bottom))
   )
-  (text "Only fan header M1 has the Tach connected.\nThe fan controller will adjust pwm only depending on the speed of M1.\nSo make sure to use M1 first\n"
-    (at 176.53 29.21 0)
+  (text "Only fan header M2 has the Tach connected.\nThe fan controller will adjust pwm only depending on the speed of M2.\nSo make sure to use M2 first. \nAlso i suggest not mixing fans \nif you are using the power pin to adjust speed.\n"
+    (at 176.53 32.385 0)
     (effects (font (size 1.27 1.27)) (justify left bottom))
   )
@@
       (effects (font (size 1.27 1.27)) (justify left top) hide)
     )
+    (property "LCSC" "" (at 146.05 74.93 0)
+      (effects (font (size 1.27 1.27)) hide)
+    )
     (pin "2")
     (pin "3")
@@
     )
     (property "Datasheet" "~" (at 69.85 36.83 0)
+      (effects (font (size 1.27 1.27)) hide)
+    )
+    (property "LCSC" "" (at 69.85 36.83 0)
       (effects (font (size 1.27 1.27)) hide)
     )
@@
       (effects (font (size 1.27 1.27)))
     )
-    (property "Value" "2KOhm" (at 139.7 33.02 90)
+    (property "Value" "2K" (at 139.7 33.02 90)
       (effects (font (size 1.27 1.27)))
     )
@@
     )
     (property "Datasheet" "~" (at 142.24 33.02 0)
+      (effects (font (size 1.27 1.27)) hide)
+    )
+    (property "LCSC" "" (at 142.24 33.02 0)
       (effects (font (size 1.27 1.27)) hide)
     )
@@
       (effects (font (size 1.27 1.27)) (justify left top) hide)
     )
+    (property "LCSC" "" (at 130.81 67.31 0)
+      (effects (font (size 1.27 1.27)) hide)
+    )
     (pin "2")
     (pin "3")
@@
       (effects (font (size 1.27 1.27)))
     )
-    (property "Value" "2KOhm" (at 74.93 53.34 90)
+    (property "Value" "2K" (at 74.93 53.34 90)
       (effects (font (size 1.27 1.27)))
     )
@@
       (effects (font (size 1.27 1.27)) hide)
     )
+    (property "LCSC" "" (at 74.93 55.88 0)
+      (effects (font (size 1.27 1.27)) hide)
+    )
     (pin "1")
     (pin "2")
@@
       (effects (font (size 1.27 1.27)) (justify left top) hide)
     )
+    (property "LCSC" "" (at 82.55 34.29 0)
+      (effects (font (size 1.27 1.27)) hide)
+    )
     (pin "8")

Commit message: V0.2 maybe
Parts:
- added R34: 10K, Resistor_SMD:R_0805_2012Metric, symbol Device:R
Connections:
- net +3.3V: now also R34.2
- net Fan1MOS: now also R34.1
Changed lines of the file:
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@@
     (title "ESPHome All in One Dev kit")
+  )
+  (junction (at 144.78 74.93) (diameter 0) (color 0 0 0 0)
   )
   (junction (at 146.05 55.88) (diameter 0) (color 0 0 0 0)
@@
     (stroke (width 0) (type default))
   )
-  (wire (pts (xy 132.08 74.93) (xy 146.05 74.93))
+  (wire (pts (xy 133.35 74.93) (xy 144.78 74.93))
     (stroke (width 0) (type default))
   )
@@
     (stroke (width 0) (type default))
   )
+  (wire (pts (xy 144.78 74.93) (xy 146.05 74.93))
+    (stroke (width 0) (type default))
+  )
   (wire (pts (xy 78.74 55.88) (xy 82.55 55.88))
     (stroke (width 0) (type default))
@@
     (stroke (width 0) (type default))
   )
+  (wire (pts (xy 144.78 74.295) (xy 144.78 74.93))
+    (stroke (width 0) (type default))
+  )
   (wire (pts (xy 120.65 34.29) (xy 123.19 34.29))
     (stroke (width 0) (type default))
@@
   )
   (wire (pts (xy 153.67 55.88) (xy 153.67 64.77))
+    (stroke (width 0) (type default))
+  )
+  (wire (pts (xy 144.78 63.5) (xy 144.78 66.675))
     (stroke (width 0) (type default))
   )
@@
     (effects (font (size 1.27 1.27)) (justify left))
   )
-  (hierarchical_label "Fan1MOS" (shape input) (at 132.08 74.93 180) (fields_autoplaced)
+  (hierarchical_label "Fan1MOS" (shape input) (at 133.35 74.93 180) (fields_autoplaced)
     (effects (font (size 1.27 1.27)) (justify right))
   )
   (hierarchical_label "SMdata" (shape input) (at 123.19 36.83 0) (fields_autoplaced)
     (effects (font (size 1.27 1.27)) (justify left))
+  )
+  (symbol (lib_id "Device:R") (at 144.78 70.485 180) (unit 1)
+    (in_bom yes) (on_board yes) (dnp no)
+    (property "Reference" "R34" (at 139.7 70.485 90)
+      (effects (font (size 1.27 1.27)))
+    )
+    (property "Value" "10K" (at 142.24 70.485 90)
+      (effects (font (size 1.27 1.27)))
+    )
+    (property "Footprint" "Resistor_SMD:R_0805_2012Metric" (at 146.558 70.485 90)
+      (effects (font (size 1.27 1.27)) hide)
+    )
+    (property "Datasheet" "~" (at 144.78 70.485 0)
+      (effects (font (size 1.27 1.27)) hide)
+    )
+    (property "LCSC" "" (at 144.78 70.485 0)
+      (effects (font (size 1.27 1.27)) hide)
+    )
+    (pin "1")
+    (pin "2")
+    (instances
+      (project "ESPHome AIO"
+        (path "/5cdf3b4f-d143-42e3-ac6f-eec5265de1fa/de469bc3-ee25-4a6a-9df7-c0a954ea29b4"
+          (reference "R34") (unit 1)
+        )
+      )
+    )
   )
   (symbol (lib_id "power:GND") (at 146.05 91.44 0) (unit 1)
@@
         )
       )
+    )
+  )
+  (symbol (lib_id "power:+3.3V") (at 144.78 63.5 0) (unit 1)
+    (in_bom yes) (on_board yes) (dnp no) (fields_autoplaced)
+    (property "Reference" "#PWR091" (at 144.78 67.31 0)
+      (effects (font (size 1.27 1.27)) hide)
+    )
+    (property "Value" "+3.3V" (at 144.78 58.42 0)
+      (effects (font (size 1.27 1.27)))
+    )
+    (property "Footprint" "" (at 144.78 63.5 0)
+      (effects (font (size 1.27 1.27)) hide)
+    )
+    (property "Datasheet" "" (at 144.78 63.5 0)
+      (effects (font (size 1.27 1.27)) hide)
+    )
+    (pin "1")
+    (instances
+      (project "ESPHome AIO"
+        (path "/5cdf3b4f-d143-42e3-ac6f-eec5265de1fa/de469bc3-ee25-4a6a-9df7-c0a954ea29b4"
+          (reference "#PWR091") (unit 1)
+        )
+      )

Commit message: V0.2 wip
Parts:
- added D6: BZX384-C5V1, ComponentSearch:SOD2512X110N, symbol ComponentSearch:BZX384-C5V1
Connections:
- net GND: now also D6.2 (A)
- net TACH: now also D6.1 (K)
Changed lines of the file:
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@@
     (title "ESPHome All in One Dev kit")
+  )
+  (junction (at 158.75 39.37) (diameter 0) (color 0 0 0 0)
   )
   (junction (at 144.78 74.93) (diameter 0) (color 0 0 0 0)
@@
     (stroke (width 0) (type default))
   )
+  (wire (pts (xy 158.75 48.26) (xy 158.75 50.165))
+    (stroke (width 0) (type default))
+  )
+  (wire (pts (xy 158.75 39.37) (xy 158.75 40.64))
+    (stroke (width 0) (type default))
+  )
   (wire (pts (xy 82.55 41.91) (xy 82.55 55.88))
     (stroke (width 0) (type default))
@@
     (stroke (width 0) (type default))
   )
+  (wire (pts (xy 158.75 39.37) (xy 167.64 39.37))
+    (stroke (width 0) (type default))
+  )
   (wire (pts (xy 250.19 36.83) (xy 257.81 36.83))
     (stroke (width 0) (type default))
@@
     (stroke (width 0) (type default))
   )
-  (wire (pts (xy 142.24 39.37) (xy 151.13 39.37))
+  (wire (pts (xy 142.24 39.37) (xy 158.75 39.37))
     (stroke (width 0) (type default))
   )
@@
     (fill (type none))
   )
-  (rectangle (start 59.69 19.05) (end 171.45 102.87)
+  (rectangle (start 59.69 19.05) (end 175.26 102.87)
     (stroke (width 0) (type dash))
     (fill (type none))
@@
   )
   (text "At 5V using 4 fans might be too much current for the mosfet.\nAt 12v you could connect way more fans.\nKeep an eye on the temprature of the mosfets."
-    (at 172.72 83.82 0)
+    (at 181.61 83.82 0)
     (effects (font (size 1.27 1.27)) (justify left bottom))
   )
@@
     (effects (font (size 1.27 1.27)) (justify left bottom))
   )
-  (text "Turn off fan1MOS for 3Pin/DC Mode" (at 172.72 67.31 0)
+  (text "Turn off fan1MOS for 3Pin/DC Mode" (at 181.61 67.31 0)
     (effects (font (size 1.27 1.27)) (justify left bottom))
   )
@@
     (effects (font (size 1.27 1.27)) (justify left bottom))
   )
-  (label "TACH" (at 151.13 39.37 180) (fields_autoplaced)
+  (label "TACH" (at 167.64 39.37 180) (fields_autoplaced)
     (effects (font (size 1.27 1.27)) (justify right bottom))
   )
@@
     )
   )
+  (symbol (lib_id "ComponentSearch:BZX384-C5V1") (at 159.385 36.195 270) (unit 1)
+    (in_bom yes) (on_board yes) (dnp no)
+    (property "Reference" "D6" (at 161.29 42.545 90)
+      (effects (font (size 1.27 1.27)) (justify left))
+    )
+    (property "Value" "BZX384-C5V1" (at 161.29 45.085 90)
+      (effects (font (size 1.27 1.27)) (justify left))
+    )
+    (property "Footprint" "ComponentSearch:SOD2512X110N" (at 61.925 47.625 0)
+      (effects (font (size 1.27 1.27)) (justify left top) hide)
+    )
+    (property "Datasheet" "https://datasheet.datasheetarchive.com/originals/distributors/Datasheets-20/DSA-380037.pdf" (at -38.075 47.625 0)
+      (effects (font (size 1.27 1.27)) (justify left top) hide)
+    )
+    (property "Height" "1.1" (at -238.075 47.625 0)
+      (effects (font (size 1.27 1.27)) (justify left top) hide)
+    )
+    (property "Manufacturer_Name" "Nexperia" (at -338.075 47.625 0)
+      (effects (font (size 1.27 1.27)) (justify left top) hide)
+    )
+    (property "Manufacturer_Part_Number" "BZX384-C5V1" (at -438.075 47.625 0)
+      (effects (font (size 1.27 1.27)) (justify left top) hide)
+    )
+    (property "Mouser Part Number" "N/A" (at -538.075 47.625 0)
+      (effects (font (size 1.27 1.27)) (justify left top) hide)
+    )
+    (property "Mouser Price/Stock" "https://www.mouser.co.uk/ProductDetail/Nexperia/BZX384-C5V1?qs=vHuUswq2%252Bszm012Dq%252BI0lA%3D%3D" (at -638.075 47.625 0)
+      (effects (font (size 1.27 1.27)) (justify left top) hide)
+    )
+    (property "Arrow Part Number" "" (at -738.075 47.625 0)
+      (effects (font (size 1.27 1.27)) (justify left top) hide)
+    )
+    (property "Arrow Price/Stock" "" (at -838.075 47.625 0)
+      (effects (font (size 1.27 1.27)) (justify left top) hide)
+    )
+    (pin "1")
+    (pin "2")
+    (instances
+      (project "ESPHome AIO"
+        (path "/5cdf3b4f-d143-42e3-ac6f-eec5265de1fa/de469bc3-ee25-4a6a-9df7-c0a954ea29b4"
+          (reference "D6") (unit 1)
+        )
+      )
+    )
+  )
   (symbol (lib_id "ComponentSearch:DMN4035L-7") (at 146.05 74.93 0) (unit 1)
     (in_bom yes) (on_board yes) (dnp no) (fields_autoplaced)
@@
         )
       )
+    )
+  )
+  (symbol (lib_id "power:GND") (at 158.75 50.165 0) (unit 1)
+    (in_bom yes) (on_board yes) (dnp no) (fields_autoplaced)
+    (property "Reference" "#PWR072" (at 158.75 56.515 0)
+      (effects (font (size 1.27 1.27)) hide)
+    )
+    (property "Value" "GND" (at 158.75 55.245 0)
+      (effects (font (size 1.27 1.27)))
+    )
+    (property "Footprint" "" (at 158.75 50.165 0)
+      (effects (font (size 1.27 1.27)) hide)
+    )
+    (property "Datasheet" "" (at 158.75 50.165 0)
+      (effects (font (size 1.27 1.27)) hide)
+    )
+    (pin "1")
+    (instances
+      (project "ESPHome AIO"
+        (path "/5cdf3b4f-d143-42e3-ac6f-eec5265de1fa/de469bc3-ee25-4a6a-9df7-c0a954ea29b4"
+          (reference "#PWR072") (unit 1)
+        )
+      )

Commit message: 0.2
Parts:
- removed Q1, Q2: DMN4035L-7, ComponentSearch:SOT96P240X110-3N, symbol ComponentSearch:DMN4035L-7
- added Q1, Q2: RQ3E080BNTB, ComponentSearch:RQ3E080BNTB, symbol ComponentSearch:RQ3E080BNTB
Connections:
- net FAN: now also Q2.4 (G)
- net Fan1MOS: now also Q1.4 (G)
- net GND: now also Q1.1 (S), Q1.2 (SOURCE_2), Q1.3 (SOURCE_3), Q2.1 (S), Q2.2 (SOURCE_2), Q2.3 (SOURCE_3)
- net MOS: now also Q1.5 (D), Q1.6 (DRAIN_2), Q1.7 (DRAIN_3), Q1.8 (DRAIN_4), Q1.9 (DRAIN_5), Q2.5 (D), Q2.6 (DRAIN_2), Q2.7 (DRAIN_3), Q2.8 (DRAIN_4), Q2.9 (DRAIN_5)
