File: KiCad Schematics and pcb/I2C.kicad_sch (KiCad schematic)
At the start: 12 parts, among them J10 Conn_01x04, J11 Conn_01x04, J12 Conn_01x04, J9 Conn_01x04, SW1 SW_DPDT_x2, SW2 SW_DPDT_x2, SW3 SW_DPDT_x2, SW4 SW_DPDT_x2, SW5 SW_DPDT_x2, SW6 SW_DPDT_x2, SW7 SW_DPDT_x2, SW8 SW_DPDT_x2

Commit message: start pcb
Parts:
- J11: renamed from J10; footprint Connector_Phoenix_MSTB:PhoenixContact_MSTBA_2,5_2-G-5,08_1x02_P5.08mm_Horizontal -> Connector_PinHeader_2.54mm:PinHeader_1x04_P2.54mm_Vertical
- renumbered J9 to J10, J11 to J12, J12 to J13, SW8 to SW10, SW1 to SW3, SW2 to SW4, SW3 to SW5, SW4 to SW6, SW5 to SW7, SW6 to SW8, SW7 to SW9

Commit message: done for the day
Parts:
- removed J12: Conn_01x04, Connector_PinHeader_2.54mm:PinHeader_1x04_P2.54mm_Vertical, symbol Connector_Generic:Conn_01x04
- removed SW7, SW9: SW_DPDT_x2, Button_Switch_THT:SW_CuK_JS202011CQN_DPDT_Straight, symbol Switch:SW_DPDT_x2

Commit message: posible V0.1
Changed lines of the file:
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@@
     (effects (font (size 1.27 1.27)) (justify left bottom))
   )
-  (global_label "I2C{slash}SMdata" (shape input) (at 116.84 22.86 0) (fields_autoplaced)
+  (hierarchical_label "I2C{slash}SMclk" (shape input) (at 246.38 114.3 0) (fields_autoplaced)
     (effects (font (size 1.27 1.27)) (justify left))
-    (property "Intersheetrefs" "${INTERSHEET_REFS}" (at 131.0736 22.86 0)
-      (effects (font (size 1.27 1.27)) (justify left) hide)
-    )
   )
-  (global_label "I2C{slash}SMclk" (shape input) (at 119.38 120.65 0) (fields_autoplaced)
+  (hierarchical_label "I2C{slash}SMclk" (shape input) (at 119.38 120.65 0) (fields_autoplaced)
     (effects (font (size 1.27 1.27)) (justify left))
-    (property "Intersheetrefs" "${INTERSHEET_REFS}" (at 132.2228 120.65 0)
-      (effects (font (size 1.27 1.27)) (justify left) hide)
-    )
   )
-  (global_label "I2C{slash}SMdata" (shape input) (at 246.38 93.98 0) (fields_autoplaced)
+  (hierarchical_label "I2C{slash}SMclk" (shape input) (at 116.84 43.18 0) (fields_autoplaced)
     (effects (font (size 1.27 1.27)) (justify left))
-    (property "Intersheetrefs" "${INTERSHEET_REFS}" (at 260.6136 93.98 0)
-      (effects (font (size 1.27 1.27)) (justify left) hide)
-    )
   )
-  (global_label "I2C{slash}SMclk" (shape input) (at 246.38 114.3 0) (fields_autoplaced)
+  (hierarchical_label "I2C{slash}SMdata" (shape input) (at 119.38 100.33 0) (fields_autoplaced)
     (effects (font (size 1.27 1.27)) (justify left))
-    (property "Intersheetrefs" "${INTERSHEET_REFS}" (at 259.2228 114.3 0)
-      (effects (font (size 1.27 1.27)) (justify left) hide)
-    )
   )
-  (global_label "I2C{slash}SMdata" (shape input) (at 119.38 100.33 0) (fields_autoplaced)
+  (hierarchical_label "I2C{slash}SMdata" (shape input) (at 116.84 22.86 0) (fields_autoplaced)
     (effects (font (size 1.27 1.27)) (justify left))
-    (property "Intersheetrefs" "${INTERSHEET_REFS}" (at 133.6136 100.33 0)
-      (effects (font (size 1.27 1.27)) (justify left) hide)
-    )
   )
-  (global_label "I2C{slash}SMclk" (shape input) (at 116.84 43.18 0) (fields_autoplaced)
+  (hierarchical_label "I2C{slash}SMdata" (shape input) (at 246.38 93.98 0) (fields_autoplaced)
     (effects (font (size 1.27 1.27)) (justify left))
-    (property "Intersheetrefs" "${INTERSHEET_REFS}" (at 129.6828 43.18 0)
-      (effects (font (size 1.27 1.27)) (justify left) hide)
-    )
   )
   (symbol (lib_id "Connector_Generic:Conn_01x04") (at 35.56 36.83 180) (unit 1)

Commit message: v0.1
Other:
- moved on the sheet: J10, J11, J13, SW10A, SW10B, SW3A, SW3B, SW4A, SW4B, SW5A, SW5B, SW6A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

Commit message: 0.2
Parts:
- SW10, SW3, SW4, SW5, SW6, SW8: footprint Button_Switch_THT:SW_CuK_JS202011CQN_DPDT_Straight -> ComponentSearch:SW_CK_JS202011CQN_DPDT_Straight
