File: KiCad Schematics and pcb/RGB.kicad_sch (KiCad schematic)
At the start: 15 parts, among them J13 Screw_Terminal_01x03, J5 Screw_Terminal_01x06, Q13 2N7002NXAKR, Q3 DMN4035L-7, Q4 DMN4035L-7, Q5 DMN4035L-7, Q6 DMN4035L-7, Q7 DMN4035L-7

Commit message: start pcb
Parts:
- J6: renamed from J13; footprint Connector_PinHeader_2.54mm:PinHeader_2x12_P2.54mm_Vertical -> Connector_Phoenix_MSTB:PhoenixContact_MSTBA_2,5_3-G-5,08_1x03_P5.08mm_Horizontal
- Q3, Q4, Q5, Q6, Q7: footprint SOT96P240X110-3N -> ComponentSearch:SOT96P240X110-3N
- Q8: renamed from Q13; footprint SOT95P230X110-3N -> ComponentSearch:SOT95P230X110-3N
- renumbered R8 to R10, R9 to R11, R28 to R12, R29 to R13, R5 to R7, R6 to R8, R7 to R9

Commit message: v0.1
Changed lines of the file:
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@@
   )
   (rectangle (start 187.96 114.3) (end 284.48 162.56)
-    (stroke (width 0) (type default))
+    (stroke (width 0) (type dash))
     (fill (type none))
   )
   (rectangle (start 12.7 12.7) (end 156.21 149.86)
-    (stroke (width 0) (type default))
+    (stroke (width 0) (type dash))
     (fill (type none))
   )

Commit message: 0.2
Parts:
- removed Q3, Q4, Q5, Q6, Q7: DMN4035L-7, ComponentSearch:SOT96P240X110-3N, symbol ComponentSearch:DMN4035L-7
- added Q3, Q4, Q5, Q6, Q7: RQ3E080BNTB, ComponentSearch:RQ3E080BNTB, symbol ComponentSearch:RQ3E080BNTB
Connections:
- net B: now also Q5.4 (G)
- net CW: now also Q6.4 (G)
- net G: now also Q4.4 (G)
- net GND: now also Q3.1 (S), Q3.2 (SOURCE_2), Q3.3 (SOURCE_3), Q4.1 (S), Q4.2 (SOURCE_2), Q4.3 (SOURCE_3), Q5.1 (S), Q5.2 (SOURCE_2), Q5.3 (SOURCE_3), Q6.1 (S), Q6.2 (SOURCE_2), Q6.3 (SOURCE_3), Q7.1 (S), Q7.2 (SOURCE_2), Q7.3 (SOURCE_3)
- net R: now also Q3.4 (G)
- net WW: now also Q7.4 (G)
- net at J5.5 (Pin_5): now also Q3.5 (D), Q3.6 (DRAIN_2), Q3.7 (DRAIN_3), Q3.8 (DRAIN_4), Q3.9 (DRAIN_5)
- net at J5.1 (Pin_1): now also Q7.5 (D), Q7.6 (DRAIN_2), Q7.7 (DRAIN_3), Q7.8 (DRAIN_4), Q7.9 (DRAIN_5)
- net at J5.4 (Pin_4): now also Q4.5 (D), Q4.6 (DRAIN_2), Q4.7 (DRAIN_3), Q4.8 (DRAIN_4), Q4.9 (DRAIN_5)
- net at J5.3 (Pin_3): now also Q5.5 (D), Q5.6 (DRAIN_2), Q5.7 (DRAIN_3), Q5.8 (DRAIN_4), Q5.9 (DRAIN_5)
- net at J5.2 (Pin_2): now also Q6.5 (D), Q6.6 (DRAIN_2), Q6.7 (DRAIN_3), Q6.8 (DRAIN_4), Q6.9 (DRAIN_5)
