File: KiCad Schematics and pcb/SignalLed.kicad_sch (KiCad schematic)
At the start: 5 parts, among them Q8 DMN4035L-7

Commit message: start pcb
Parts:
- Q9: renamed from Q8; footprint SOT96P240X110-3N -> ComponentSearch:SOT96P240X110-3N
- renumbered R13 to R17, R14 to R18, R15 to R19
Changed lines of the file:
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@@
   (symbol (lib_id "Device:R") (at 35.56 39.37 0) (unit 1)
     (in_bom yes) (on_board yes) (dnp no) (fields_autoplaced)
-    (property "Reference" "R13" (at 38.1 38.1 0)
+    (property "Reference" "R17" (at 38.1 38.1 0)
       (effects (font (size 1.27 1.27)) (justify left))
     )
@@
       (project "ESPHome AIO"
         (path "/5cdf3b4f-d143-42e3-ac6f-eec5265de1fa/f403fb1f-6c3a-4b91-96f2-7610e89c4ca7/14978f3b-9ae2-49c9-8e6c-da58eba4429f"
-          (reference "R13") (unit 1)
+          (reference "R17") (unit 1)
         )
         (path "/5cdf3b4f-d143-42e3-ac6f-eec5265de1fa/f403fb1f-6c3a-4b91-96f2-7610e89c4ca7/823cca60-66a1-4835-8923-025a3c75e353"
-          (reference "R16") (unit 1)
-        )
-        (path "/5cdf3b4f-d143-42e3-ac6f-eec5265de1fa/f403fb1f-6c3a-4b91-96f2-7610e89c4ca7/d212efe7-a37c-4de7-b2c8-e89c3950f34a"
-          (reference "R19") (unit 1)
-        )
-        (path "/5cdf3b4f-d143-42e3-ac6f-eec5265de1fa/f403fb1f-6c3a-4b91-96f2-7610e89c4ca7/0dddecc0-8468-4437-9a16-5f57fc4e73e0"
-          (reference "R22") (unit 1)
+          (reference "R20") (unit 1)
         )
         (path "/5cdf3b4f-d143-42e3-ac6f-eec5265de1fa/f403fb1f-6c3a-4b91-96f2-7610e89c4ca7/0559229c-b64b-4326-a312-6c5673a85522"
-          (reference "R25") (unit 1)
+          (reference "R29") (unit 1)
         )
       )
@@
           (reference "D3") (unit 1)
         )
-        (path "/5cdf3b4f-d143-42e3-ac6f-eec5265de1fa/f403fb1f-6c3a-4b91-96f2-7610e89c4ca7/d212efe7-a37c-4de7-b2c8-e89c3950f34a"
-          (reference "D4") (unit 1)
-        )
-        (path "/5cdf3b4f-d143-42e3-ac6f-eec5265de1fa/f403fb1f-6c3a-4b91-96f2-7610e89c4ca7/0dddecc0-8468-4437-9a16-5f57fc4e73e0"
-          (reference "D5") (unit 1)
-        )
         (path "/5cdf3b4f-d143-42e3-ac6f-eec5265de1fa/f403fb1f-6c3a-4b91-96f2-7610e89c4ca7/0559229c-b64b-4326-a312-6c5673a85522"
           (reference "D6") (unit 1)
@@
   (symbol (lib_id "Device:R") (at 59.69 40.64 0) (unit 1)
     (in_bom yes) (on_board yes) (dnp no) (fields_autoplaced)
-    (property "Reference" "R15" (at 62.23 39.37 0)
+    (property "Reference" "R19" (at 62.23 39.37 0)
       (effects (font (size 1.27 1.27)) (justify left))
     )
@@
       (project "ESPHome AIO"
         (path "/5cdf3b4f-d143-42e3-ac6f-eec5265de1fa/f403fb1f-6c3a-4b91-96f2-7610e89c4ca7/14978f3b-9ae2-49c9-8e6c-da58eba4429f"
-          (reference "R15") (unit 1)
+          (reference "R19") (unit 1)
         )
         (path "/5cdf3b4f-d143-42e3-ac6f-eec5265de1fa/f403fb1f-6c3a-4b91-96f2-7610e89c4ca7/823cca60-66a1-4835-8923-025a3c75e353"
-          (reference "R18") (unit 1)
-        )
-        (path "/5cdf3b4f-d143-42e3-ac6f-eec5265de1fa/f403fb1f-6c3a-4b91-96f2-7610e89c4ca7/d212efe7-a37c-4de7-b2c8-e89c3950f34a"
-          (reference "R21") (unit 1)
-        )
-        (path "/5cdf3b4f-d143-42e3-ac6f-eec5265de1fa/f403fb1f-6c3a-4b91-96f2-7610e89c4ca7/0dddecc0-8468-4437-9a16-5f57fc4e73e0"
-          (reference "R24") (unit 1)
+          (reference "R22") (unit 1)
         )
         (path "/5cdf3b4f-d143-42e3-ac6f-eec5265de1fa/f403fb1f-6c3a-4b91-96f2-7610e89c4ca7/0559229c-b64b-4326-a312-6c5673a85522"
-          (reference "R27") (unit 1)
+          (reference "R31") (unit 1)
         )
       )
@@
   (symbol (lib_id "power:GND") (at 59.69 64.77 0) (unit 1)
     (in_bom yes) (on_board yes) (dnp no) (fields_autoplaced)
-    (property "Reference" "#PWR051" (at 59.69 71.12 0)
+    (property "Reference" "#PWR064" (at 59.69 71.12 0)
       (effects (font (size 1.27 1.27)) hide)
     )
@@
       (project "ESPHome AIO"
         (path "/5cdf3b4f-d143-42e3-ac6f-eec5265de1fa/f403fb1f-6c3a-4b91-96f2-7610e89c4ca7/14978f3b-9ae2-49c9-8e6c-da58eba4429f"
-          (reference "#PWR051") (unit 1)
+          (reference "#PWR064") (unit 1)
         )
         (path "/5cdf3b4f-d143-42e3-ac6f-eec5265de1fa/f403fb1f-6c3a-4b91-96f2-7610e89c4ca7/823cca60-66a1-4835-8923-025a3c75e353"
-          (reference "#PWR052") (unit 1)
-        )
-        (path "/5cdf3b4f-d143-42e3-ac6f-eec5265de1fa/f403fb1f-6c3a-4b91-96f2-7610e89c4ca7/d212efe7-a37c-4de7-b2c8-e89c3950f34a"
-          (reference "#PWR053") (unit 1)
-        )
-        (path "/5cdf3b4f-d143-42e3-ac6f-eec5265de1fa/f403fb1f-6c3a-4b91-96f2-7610e89c4ca7/0dddecc0-8468-4437-9a16-5f57fc4e73e0"
-          (reference "#PWR054") (unit 1)
+          (reference "#PWR065") (unit 1)
         )
         (path "/5cdf3b4f-d143-42e3-ac6f-eec5265de1fa/f403fb1f-6c3a-4b91-96f2-7610e89c4ca7/0559229c-b64b-4326-a312-6c5673a85522"
-          (reference "#PWR055") (unit 1)
+          (reference "#PWR068") (unit 1)
         )
       )
@@
   (symbol (lib_id "ComponentSearch:DMN4035L-7") (at 52.07 57.15 0) (unit 1)
     (in_bom yes) (on_board yes) (dnp no) (fields_autoplaced)
-    (property "Reference" "Q8" (at 63.5 53.34 0)
+    (property "Reference" "Q9" (at 63.5 53.34 0)
       (effects (font (size 1.27 1.27)) (justify left))
     )
@@
       (effects (font (size 1.27 1.27)) (justify left))
     )
-    (property "Footprint" "SOT96P240X110-3N" (at 63.5 155.88 0)
+    (property "Footprint" "ComponentSearch:SOT96P240X110-3N" (at 63.5 155.88 0)
       (effects (font (size 1.27 1.27)) (justify left top) hide)
     )
@@
       (project "ESPHome AIO"
         (path "/5cdf3b4f-d143-42e3-ac6f-eec5265de1fa/f403fb1f-6c3a-4b91-96f2-7610e89c4ca7/14978f3b-9ae2-49c9-8e6c-da58eba4429f"
-          (reference "Q8") (unit 1)
+          (reference "Q9") (unit 1)
         )
         (path "/5cdf3b4f-d143-42e3-ac6f-eec5265de1fa/f403fb1f-6c3a-4b91-96f2-7610e89c4ca7/823cca60-66a1-4835-8923-025a3c75e353"
-          (reference "Q9") (unit 1)
-        )
-        (path "/5cdf3b4f-d143-42e3-ac6f-eec5265de1fa/f403fb1f-6c3a-4b91-96f2-7610e89c4ca7/d212efe7-a37c-4de7-b2c8-e89c3950f34a"
           (reference "Q10") (unit 1)
         )
-        (path "/5cdf3b4f-d143-42e3-ac6f-eec5265de1fa/f403fb1f-6c3a-4b91-96f2-7610e89c4ca7/0dddecc0-8468-4437-9a16-5f57fc4e73e0"
-          (reference "Q11") (unit 1)
-        )
         (path "/5cdf3b4f-d143-42e3-ac6f-eec5265de1fa/f403fb1f-6c3a-4b91-96f2-7610e89c4ca7/0559229c-b64b-4326-a312-6c5673a85522"
-          (reference "Q12") (unit 1)
+          (reference "Q13") (unit 1)
         )
       )
@@
   (symbol (lib_id "Device:R") (at 45.72 57.15 90) (unit 1)
     (in_bom yes) (on_board yes) (dnp no) (fields_autoplaced)
-    (property "Reference" "R14" (at 45.72 50.8 90)
+    (property "Reference" "R18" (at 45.72 50.8 90)
       (effects (font (size 1.27 1.27)))
     )
@@
       (project "ESPHome AIO"
         (path "/5cdf3b4f-d143-42e3-ac6f-eec5265de1fa/f403fb1f-6c3a-4b91-96f2-7610e89c4ca7/14978f3b-9ae2-49c9-8e6c-da58eba4429f"
-          (reference "R14") (unit 1)
+          (reference "R18") (unit 1)
         )
         (path "/5cdf3b4f-d143-42e3-ac6f-eec5265de1fa/f403fb1f-6c3a-4b91-96f2-7610e89c4ca7/823cca60-66a1-4835-8923-025a3c75e353"
-          (reference "R17") (unit 1)
-        )
-        (path "/5cdf3b4f-d143-42e3-ac6f-eec5265de1fa/f403fb1f-6c3a-4b91-96f2-7610e89c4ca7/d212efe7-a37c-4de7-b2c8-e89c3950f34a"
-          (reference "R20") (unit 1)
-        )
-        (path "/5cdf3b4f-d143-42e3-ac6f-eec5265de1fa/f403fb1f-6c3a-4b91-96f2-7610e89c4ca7/0dddecc0-8468-4437-9a16-5f57fc4e73e0"
-          (reference "R23") (unit 1)
+          (reference "R21") (unit 1)
         )
         (path "/5cdf3b4f-d143-42e3-ac6f-eec5265de1fa/f403fb1f-6c3a-4b91-96f2-7610e89c4ca7/0559229c-b64b-4326-a312-6c5673a85522"
-          (reference "R26") (unit 1)
+          (reference "R30") (unit 1)
         )
       )

Commit message: v0.1
Other:
- note added: "Mosfet LED driver"
Changed lines of the file:
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@@
     (stroke (width 0) (type default))
+  )
+  (rectangle (start 22.86 20.32) (end 78.74 73.66)
+    (stroke (width 0) (type dash))
+    (fill (type none))
+  )
+  (text "Mosfet LED driver" (at 22.86 20.32 0)
+    (effects (font (size 1.27 1.27)) (justify left bottom))
   )
   (hierarchical_label "GPIO" (shape input) (at 30.48 57.15 180) (fields_autoplaced)

Commit message: V0.2 maybe
Parts:
- removed Q9: DMN4035L-7, ComponentSearch:SOT96P240X110-3N, symbol ComponentSearch:DMN4035L-7
- added Q12: 2N7002NXAKR, SOT95P230X110-3N, symbol ComponentSearch:2N7002NXAKR
Connections:
- net GND: now also Q12.2 (S)
- net at R19.2: now also Q12.3 (D)
- net at R18.2: now also Q12.1 (G)
Changed lines of the file:
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@@
-    )
-  )
-  (symbol (lib_id "ComponentSearch:DMN4035L-7") (at 52.07 57.15 0) (unit 1)
-    (in_bom yes) (on_board yes) (dnp no) (fields_autoplaced)
-    (property "Reference" "Q9" (at 63.5 53.34 0)
-      (effects (font (size 1.27 1.27)) (justify left))
-    )
-    (property "Value" "DMN4035L-7" (at 63.5 55.88 0)
-      (effects (font (size 1.27 1.27)) (justify left))
-    )
-    (property "Footprint" "ComponentSearch:SOT96P240X110-3N" (at 63.5 155.88 0)
-      (effects (font (size 1.27 1.27)) (justify left top) hide)
-    )
-    (property "Datasheet" "https://www.diodes.com/assets/Datasheets/DMN2310U.pdf" (at 63.5 255.88 0)
-      (effects (font (size 1.27 1.27)) (justify left top) hide)
-    )
-    (property "Height" "1.1" (at 63.5 455.88 0)
-      (effects (font (size 1.27 1.27)) (justify left top) hide)
-    )
-    (property "Manufacturer_Name" "Diodes Incorporated" (at 63.5 555.88 0)
-      (effects (font (size 1.27 1.27)) (justify left top) hide)
-    )
-    (property "Manufacturer_Part_Number" "DMN4035L-7" (at 63.5 655.88 0)
-      (effects (font (size 1.27 1.27)) (justify left top) hide)
-    )
-    (property "Mouser Part Number" "621-DMN4035L-7" (at 63.5 755.88 0)
-      (effects (font (size 1.27 1.27)) (justify left top) hide)
-    )
-    (property "Mouser Price/Stock" "https://www.mouser.co.uk/ProductDetail/Diodes-Incorporated/DMN2310U-7?qs=xZ%2FP%252Ba9zWqY%252BAdKLxIytvQ%3D%3D" (at 63.5 855.88 0)
-      (effects (font (size 1.27 1.27)) (justify left top) hide)
-    )
-    (property "Arrow Part Number" "" (at 63.5 955.88 0)
-      (effects (font (size 1.27 1.27)) (justify left top) hide)
-    )
-    (property "Arrow Price/Stock" "" (at 63.5 1055.88 0)
-      (effects (font (size 1.27 1.27)) (justify left top) hide)
-    )
-    (property "LCSC" "" (at 52.07 57.15 0)
-      (effects (font (size 1.27 1.27)) hide)
-    )
-    (pin "2")
-    (pin "3")
-    (pin "1")
-    (instances
-      (project "ESPHome AIO"
-        (path "/5cdf3b4f-d143-42e3-ac6f-eec5265de1fa/f403fb1f-6c3a-4b91-96f2-7610e89c4ca7/14978f3b-9ae2-49c9-8e6c-da58eba4429f"
-          (reference "Q9") (unit 1)
-        )
-        (path "/5cdf3b4f-d143-42e3-ac6f-eec5265de1fa/f403fb1f-6c3a-4b91-96f2-7610e89c4ca7/d9e01f38-4d9f-440d-a1ac-085be380d734"
-          (reference "Q10") (unit 1)
-        )
-      )
     )
   )
@@
         )
       )
+    )
+  )
+  (symbol (lib_id "ComponentSearch:2N7002NXAKR") (at 52.07 57.15 0) (unit 1)
+    (in_bom yes) (on_board yes) (dnp no) (fields_autoplaced)
+    (property "Reference" "Q12" (at 63.5 53.34 0)
+      (effects (font (size 1.27 1.27)) (justify left))
+    )
+    (property "Value" "2N7002NXAKR" (at 63.5 55.88 0)
+      (effects (font (size 1.27 1.27)) (justify left))
+    )
+    (property "Footprint" "SOT95P230X110-3N" (at 63.5 155.88 0)
+      (effects (font (size 1.27 1.27)) (justify left top) hide)
+    )
+    (property "Datasheet" "https://assets.nexperia.com/documents/data-sheet/2N7002NXAK.pdf" (at 63.5 255.88 0)
+      (effects (font (size 1.27 1.27)) (justify left top) hide)
+    )
+    (property "Height" "1.1" (at 63.5 455.88 0)
+      (effects (font (size 1.27 1.27)) (justify left top) hide)
+    )
+    (property "Manufacturer_Name" "Nexperia" (at 63.5 555.88 0)
+      (effects (font (size 1.27 1.27)) (justify left top) hide)
+    )
+    (property "Manufacturer_Part_Number" "2N7002NXAKR" (at 63.5 655.88 0)
+      (effects (font (size 1.27 1.27)) (justify left top) hide)
+    )
+    (property "Mouser Part Number" "771-2N7002NXAKR" (at 63.5 755.88 0)
+      (effects (font (size 1.27 1.27)) (justify left top) hide)
+    )
+    (property "Mouser Price/Stock" "https://www.mouser.co.uk/ProductDetail/Nexperia/2N7002NXAKR?qs=%252B6g0mu59x7JoAsZYPFXqhw%3D%3D" (at 63.5 855.88 0)
+      (effects (font (size 1.27 1.27)) (justify left top) hide)
+    )
+    (property "Arrow Part Number" "2N7002NXAKR" (at 63.5 955.88 0)
+      (effects (font (size 1.27 1.27)) (justify left top) hide)
+    )
+    (property "Arrow Price/Stock" "https://www.arrow.com/en/products/2n7002nxakr/nexperia?region=europe" (at 63.5 1055.88 0)
+      (effects (font (size 1.27 1.27)) (justify left top) hide)
+    )
+    (pin "1")
+    (pin "2")
+    (pin "3")
+    (instances
+      (project "ESPHome AIO"
+        (path "/5cdf3b4f-d143-42e3-ac6f-eec5265de1fa/f403fb1f-6c3a-4b91-96f2-7610e89c4ca7/d9e01f38-4d9f-440d-a1ac-085be380d734"
+          (reference "Q12") (unit 1)
+        )
+        (path "/5cdf3b4f-d143-42e3-ac6f-eec5265de1fa/f403fb1f-6c3a-4b91-96f2-7610e89c4ca7/14978f3b-9ae2-49c9-8e6c-da58eba4429f"
+          (reference "Q11") (unit 1)
+        )
+      )

Commit message: V0.2 wip
Parts:
- Q12: footprint SOT95P230X110-3N -> ComponentSearch:SOT95P230X110-3N
Changed lines of the file:
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@@
       (effects (font (size 1.27 1.27)) (justify left))
     )
-    (property "Footprint" "SOT95P230X110-3N" (at 63.5 155.88 0)
+    (property "Footprint" "ComponentSearch:SOT95P230X110-3N" (at 63.5 155.88 0)
       (effects (font (size 1.27 1.27)) (justify left top) hide)
     )

Commit message: 0.2
Parts:
- R17: value 11K -> 10K
- R19: value 33K -> 10K
- renumbered Q12 to Q11
