File: KiCad Schematics and pcb/power.kicad_sch (KiCad schematic)
At the start: 11 parts, among them IC4 LD1085D2T33R, IC5 BD50FC0FP-E2, J7 Screw_Terminal_01x02, J8 694106301002

Commit message: start pcb
Parts:
- IC5: renamed from IC4; footprint LD1085D2T33R -> ComponentSearch:LD1085D2T33R
- IC6: renamed from IC5; footprint BD50FC0FPE2 -> ComponentSearch:BD50FC0FPE2
- J8: renamed from J7; footprint ComponentSearch:694106301002_1 -> Connector_Phoenix_MSTB:PhoenixContact_MSTBA_2,5_2-G-5,08_1x02_P5.08mm_Horizontal
- J9: renamed from J8; footprint 694106301002_1 -> ComponentSearch:694106301002_1

Commit message: v0.1 prototype ordered
Parts:
- added D4, D5: LED, LED_SMD:LED_0805_2012Metric, symbol Device:LED
- added IC7: BZX84-C12, ComponentSearch:SOT95P230X110-3N, symbol ComponentSearch:BZX84-C12
- added IC8, IC9: TPS259573DSGR, ComponentSearch:SON50P200X200X80-9N, symbol ComponentSearch:TPS259573DSGR
- added JP2: SolderJumper_2_Bridged, Jumper:SolderJumper-2_P1.3mm_Open_TrianglePad1.0x1.5mm, symbol Jumper:SolderJumper_2_Bridged
- added JP3: Jumper_3_Bridged12, Connector_PinHeader_2.54mm:PinHeader_1x03_P2.54mm_Vertical, symbol Jumper:Jumper_3_Bridged12
- added R23, R31: 10K, Resistor_SMD:R_0805_2012Metric, symbol Device:R
- added R24: 36.5K, Resistor_SMD:R_0805_2012Metric, symbol Device:R
- added R25: 2.32K, Resistor_SMD:R_0805_2012Metric, symbol Device:R
- added R26: 2.2K, Resistor_SMD:R_0805_2012Metric, symbol Device:R
- added R27: 1K, Resistor_SMD:R_0805_2012Metric, symbol Device:R
- added R28: 487, Resistor_SMD:R_0805_2012Metric, symbol Device:R
- added R29: 715, Resistor_SMD:R_0805_2012Metric, symbol Device:R
- added R30: 20.5K, Resistor_SMD:R_0805_2012Metric, symbol Device:R
- added R32: 680, Resistor_SMD:R_0805_2012Metric, symbol Device:R
- F1: footprint Fuse:Fuseholder_Clip-5x20mm_Bel_FC-203-22_Lateral_P17.80x5.00mm_D1.17mm_Horizontal -> Fuse:Fuseholder_Littelfuse_Nano2_154x
- J9: value 694106301002 -> XKB Connection DC-005-5A-3.0; footprint ComponentSearch:694106301002_1 -> Connector_BarrelJack:BarrelJack_Horizontal
Connections:
- net +3.3V: now also IC9.5 (OUT); no longer C13.1, IC5.4 (OUTPUT)
- net +5V: now also IC8.5 (OUT); no longer C12.1, IC6.3 (VO), JP1.2 (B)
- net GND: now also IC7.1 (A), IC8.8 (GND_1), IC8.9 (GND_2), IC9.8 (GND_1), IC9.9 (GND_2), R23.2, R25.2, R27.2, R28.2, R29.2, R31.2
- new net: C13.1, IC5.4 (OUTPUT), IC9.3 (IN_1), IC9.4 (IN_2), R30.1, R32.1
- new net: IC7.3 (K), IC8.3 (IN_1), IC8.4 (IN_2), JP1.2 (B), JP2.2 (B), R24.1, R26.1
- new net: JP3.1 (A), R25.1
- new net: IC9.2 (~{EN}/OVLO), R30.2, R31.1
- new net: D5.2 (A), R32.2
- new net: D4.2 (A), R26.2, R27.1
- new net: D5.1 (K), IC9.6 (~{FLT})
- new net: C12.1, IC6.3 (VO), JP2.1 (A)
- new net: IC8.2 (~{EN}/OVLO), R23.1, R24.2
- new net: IC9.7 (ILM), R29.1
- new net: D4.1 (K), IC8.6 (~{FLT})
- new net: IC8.7 (ILM), JP3.2 (C)
- new net: JP3.3 (B), R28.1
- no-connect marks 0 -> 2
Other:
- note added: "All resistor values are calculated to garantee function with a 1% tollerance"
- note added: "Be carefull with these jumpers. If you do not cut jp2 when connecting jp1 you might break the 5V regulator."
- note added: "Turn off worst case (low) 5.129V and (high) 5.947V with 1% resistors center = 5.538V"
- note added: "with a margin of 0.07A and a 1% resistor R25 the max current will be 910.78mA R28 is set to 4A max for the electronic fuse"
- moved on the sheet: C11, C12, IC6, JP1

Commit message: V0.2 maybe
Parts:
- removed R27: 1K, Resistor_SMD:R_0805_2012Metric, symbol Device:R
- added Q9: 2N7002NXAKR, SOT95P230X110-3N, symbol ComponentSearch:2N7002NXAKR
Connections:
- net 3.3V_FLT: now reaches D5.2 (A), R32.2
- net 3.3V_FLT: now also Q9.1 (G)
- net at IC8.2 (~{EN}/OVLO), R24.2: now also Q9.3 (D); no longer R23.1
- new net: Q9.2 (S), R23.1
Other:
- moved on the sheet: R23, R26, R29

Commit message: V0.2 wip
Parts:
- J9: footprint Connector_BarrelJack:BarrelJack_Horizontal -> ComponentSearch:694106301002_1
- Q9: footprint SOT95P230X110-3N -> ComponentSearch:SOT95P230X110-3N
Connections:
- net 3.3V_FLT: now also D5.1 (K), IC9.6 (~{FLT}); no longer D5.2 (A), R32.2
- net 5V-24V: no longer C10.1, IC5.3 (INPUT)
- new net: D5.2 (A), R32.2
- new net VBUS: C10.1, IC5.3 (INPUT)
Other:
- note added: "3.3V straigt to vbus"
- note added: "with a margin of 0.07A and a 1% resistor R25 the max current will be 910.78mA R28 is set to 4A max for the electronic fuse. Move jumper when using an external 5V suply capable of suplying more than 1A If you need more than 4A on 5V rail change resistor acording to the datasheet. R28 is a suggestion for a 4A limit sparing your replacable fuse."
- note removed: "with a margin of 0.07A and a 1% resistor R25 the max current will be 910.78mA R28 is set to 4A max for the electronic fuse"
Changed lines of the file:
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@@
   (junction (at 103.505 151.13) (diameter 0) (color 0 0 0 0)
   )
+  (junction (at 150.495 114.935) (diameter 0) (color 0 0 0 0)
+  )
   (junction (at 59.69 173.99) (diameter 0) (color 0 0 0 0)
   )
@@
   )
   (junction (at 20.32 38.1) (diameter 0) (color 0 0 0 0)
-  )
-  (junction (at 146.05 128.905) (diameter 0) (color 0 0 0 0)
   )
   (no_connect (at 111.125 105.41))
@@
     (stroke (width 0) (type default))
   )
-  (wire (pts (xy 154.94 128.905) (xy 146.05 128.905))
-    (stroke (width 0) (type default))
-  )
   (wire (pts (xy 83.82 43.18) (xy 76.2 43.18))
     (stroke (width 0) (type default))
@@
     (stroke (width 0) (type default))
   )
+  (wire (pts (xy 157.48 114.935) (xy 150.495 114.935))
+    (stroke (width 0) (type default))
+  )
   (wire (pts (xy 20.955 154.94) (xy 37.465 154.94))
     (stroke (width 0) (type default))
@@
     (stroke (width 0) (type default))
   )
+  (wire (pts (xy 46.355 109.22) (xy 49.53 109.22))
+    (stroke (width 0) (type default))
+  )
   (wire (pts (xy 167.005 113.03) (xy 167.005 101.6))
     (stroke (width 0) (type default))
@@
     (stroke (width 0) (type default))
   )
+  (wire (pts (xy 59.69 185.42) (xy 59.69 189.23))
+    (stroke (width 0) (type default))
+  )
   (wire (pts (xy 85.09 120.65) (xy 85.09 123.19))
     (stroke (width 0) (type default))
   )
-  (wire (pts (xy 49.53 102.87) (xy 49.53 109.22))
-    (stroke (width 0) (type default))
-  )
   (wire (pts (xy 82.55 109.22) (xy 85.09 109.22))
     (stroke (width 0) (type default))
@@
     (stroke (width 0) (type default))
   )
+  (wire (pts (xy 157.48 124.46) (xy 157.48 114.935))
+    (stroke (width 0) (type default))
+  )
   (wire (pts (xy 108.585 97.79) (xy 98.425 97.79))
     (stroke (width 0) (type default))
@@
     (stroke (width 0) (type default))
   )
-  (wire (pts (xy 59.69 173.99) (xy 59.69 176.53))
+  (wire (pts (xy 59.69 173.99) (xy 59.69 177.8))
     (stroke (width 0) (type default))
   )
@@
     (effects (font (size 1.27 1.27)) (justify left bottom))
   )
-  (text "with a margin of 0.07A and a 1% resistor R25 the max current will be 910.78mA\nR28 is set to 4A max for the electronic fuse"
+  (text "with a margin of 0.07A and a 1% resistor R25 the max current will be 910.78mA\nR28 is set to 4A max for the electronic fuse.\nMove jumper when using an external 5V suply capable of suplying more than 1A\nIf you need more than 4A on 5V rail change resistor acording to the datasheet.\nR28 is a suggestion for a 4A limit sparing your replacable fuse.\n"
     (at 177.165 156.845 0)
     (effects (font (size 1.27 1.27)) (justify left bottom))
@@
     (effects (font (size 1.27 1.27)) (justify left bottom))
   )
+  (text "3.3V straigt to vbus " (at 26.035 105.41 0)
+    (effects (font (size 1.27 1.27)) (justify left bottom))
+  )
   (text "5V Regulator skip if you \nuse 5v external power supply.\n"
     (at 21.59 181.61 0)
@@
     (effects (font (size 1.27 1.27)) (justify left bottom))
   )
-  (label "3.3V_FLT" (at 154.94 128.905 180) (fields_autoplaced)
-    (effects (font (size 1.27 1.27)) (justify right bottom))
+  (label "3.3V_FLT" (at 157.48 124.46 90) (fields_autoplaced)
+    (effects (font (size 1.27 1.27)) (justify left bottom))
+  )
+  (hierarchical_label "VBUS" (shape input) (at 46.355 109.22 180) (fields_autoplaced)
+    (effects (font (size 1.27 1.27)) (justify right))
   )
   (hierarchical_label "USB_PD_POWER" (shape input) (at 46.99 22.86 180) (fields_autoplaced)
@@
     )
   )
-  (symbol (lib_id "ComponentSearch:BZX84-C12") (at 59.69 170.18 270) (unit 1)
-    (in_bom yes) (on_board yes) (dnp no) (fields_autoplaced)
-    (property "Reference" "IC7" (at 62.23 181.61 90)
-      (effects (font (size 1.27 1.27)) (justify left))
-    )
-    (property "Value" "BZX84-C12" (at 62.23 184.15 90)
-      (effects (font (size 1.27 1.27)) (justify left))
-    )
-    (property "Footprint" "ComponentSearch:SOT95P230X110-3N" (at -35.23 191.77 0)
-      (effects (font (size 1.27 1.27)) (justify left top) hide)
-    )
-    (property "Datasheet" "https://assets.nexperia.com/documents/data-sheet/BZX84_SER.pdf" (at -135.23 191.77 0)
-      (effects (font (size 1.27 1.27)) (justify left top) hide)
-    )
-    (property "Height" "1.1" (at -335.23 191.77 0)
-      (effects (font (size 1.27 1.27)) (justify left top) hide)
-    )
-    (property "Manufacturer_Name" "Nexperia" (at -435.23 191.77 0)
-      (effects (font (size 1.27 1.27)) (justify left top) hide)
-    )
-    (property "Manufacturer_Part_Number" "BZX84-C12" (at -535.23 191.77 0)
-      (effects (font (size 1.27 1.27)) (justify left top) hide)
-    )
-    (property "Mouser Part Number" "N/A" (at -635.23 191.77 0)
-      (effects (font (size 1.27 1.27)) (justify left top) hide)
-    )
-    (property "Mouser Price/Stock" "https://www.mouser.co.uk/ProductDetail/Nexperia/BZX84-C12?qs=vHuUswq2%252BsxJg6DRQk2zTw%3D%3D" (at -735.23 191.77 0)
-      (effects (font (size 1.27 1.27)) (justify left top) hide)
-    )
-    (property "Arrow Part Number" "" (at -835.23 191.77 0)
-      (effects (font (size 1.27 1.27)) (justify left top) hide)
-    )
-    (property "Arrow Price/Stock" "" (at -935.23 191.77 0)
-      (effects (font (size 1.27 1.27)) (justify left top) hide)
-    )
-    (property "LCSC" "" (at 59.69 170.18 0)
+  (symbol (lib_id "ComponentSearch:BZX84-C12") (at 59.69 167.005 270) (unit 1)
+    (in_bom yes) (on_board yes) (dnp no) (fields_autoplaced)
+    (property "Reference" "IC7" (at 62.23 178.435 90)
+      (effects (font (size 1.27 1.27)) (justify left))
+    )
+    (property "Value" "BZX84-C12" (at 62.23 180.975 90)
+      (effects (font (size 1.27 1.27)) (justify left))
+    )
+    (property "Footprint" "ComponentSearch:SOT95P230X110-3N" (at -35.23 188.595 0)
+      (effects (font (size 1.27 1.27)) (justify left top) hide)
+    )
+    (property "Datasheet" "https://assets.nexperia.com/documents/data-sheet/BZX84_SER.pdf" (at -135.23 188.595 0)
+      (effects (font (size 1.27 1.27)) (justify left top) hide)
+    )
+    (property "Height" "1.1" (at -335.23 188.595 0)
+      (effects (font (size 1.27 1.27)) (justify left top) hide)
+    )
+    (property "Manufacturer_Name" "Nexperia" (at -435.23 188.595 0)
+      (effects (font (size 1.27 1.27)) (justify left top) hide)
+    )
+    (property "Manufacturer_Part_Number" "BZX84-C12" (at -535.23 188.595 0)
+      (effects (font (size 1.27 1.27)) (justify left top) hide)
+    )
+    (property "Mouser Part Number" "N/A" (at -635.23 188.595 0)
+      (effects (font (size 1.27 1.27)) (justify left top) hide)
+    )
+    (property "Mouser Price/Stock" "https://www.mouser.co.uk/ProductDetail/Nexperia/BZX84-C12?qs=vHuUswq2%252BsxJg6DRQk2zTw%3D%3D" (at -735.23 188.595 0)
+      (effects (font (size 1.27 1.27)) (justify left top) hide)
+    )
+    (property "Arrow Part Number" "" (at -835.23 188.595 0)
+      (effects (font (size 1.27 1.27)) (justify left top) hide)
+    )
+    (property "Arrow Price/Stock" "" (at -935.23 188.595 0)
+      (effects (font (size 1.27 1.27)) (justify left top) hide)
+    )
+    (property "LCSC" "" (at 59.69 167.005 0)
       (effects (font (size 1.27 1.27)) hide)
     )
@@
         (path "/5cdf3b4f-d143-42e3-ac6f-eec5265de1fa/cf8c527b-4fc6-4a23-a706-c7060e10c8ba"
           (reference "R30") (unit 1)
-        )
-      )
-    )
-  )
-  (symbol (lib_id "ComponentSearch:5V-24V") (at 49.53 102.87 0) (unit 1)
-    (in_bom yes) (on_board yes) (dnp no) (fields_autoplaced)
-    (property "Reference" "#PWR072" (at 49.53 106.68 0)
-      (effects (font (size 1.27 1.27)) hide)
-    )
-    (property "Value" "5V-24V" (at 49.53 97.79 0)
-      (effects (font (size 1.27 1.27)))
-    )
-    (property "Footprint" "" (at 49.53 102.87 0)
-      (effects (font (size 1.27 1.27)) hide)
-    )
-    (property "Datasheet" "" (at 49.53 102.87 0)
-      (effects (font (size 1.27 1.27)) hide)
-    )
-    (pin "1")
-    (instances
-      (project "ESPHome AIO"
-        (path "/5cdf3b4f-d143-42e3-ac6f-eec5265de1fa/cf8c527b-4fc6-4a23-a706-c7060e10c8ba"
-          (reference "#PWR072") (unit 1)
         )
       )
@@
       (effects (font (size 1.27 1.27)) (justify left))
     )
-    (property "Footprint" "SOT95P230X110-3N" (at 107.315 262.56 0)
+    (property "Footprint" "ComponentSearch:SOT95P230X110-3N" (at 107.315 262.56 0)
       (effects (font (size 1.27 1.27)) (justify left top) hide)
     )
@@
     )
   )
-  (symbol (lib_id "ComponentSearch:TPS259573DSGR") (at 112.395 148.59 0) (unit 1)
+  (symbol (lib_name "TPS259573DSGR_1") (lib_id "ComponentSearch:TPS259573DSGR") (at 112.395 148.59 0) (unit 1)
     (in_bom yes) (on_board yes) (dnp no) (fields_autoplaced)
     (property "Reference" "IC8" (at 130.175 140.97 0)
@@
       (effects (font (size 1.27 1.27)))
     )
-    (property "Footprint" "Connector_BarrelJack:BarrelJack_Horizontal" (at 26.67 -56.82 0)
-      (effects (font (size 1.27 1.27)) (justify left top) hide)
-    )
+    (property "Footprint" "ComponentSearch:694106301002_1" (at 26.67 -56.82 0)
+      (effects (font (size 1.27 1.27)) (justify left top) hide)
+    )

Commit message: 0.2
Parts:
- J9: footprint ComponentSearch:694106301002_1 -> Connector_BarrelJack:BarrelJack_Horizontal
Connections:
- net VBUS is gone; now on net 5V-24V: C10.1, IC5.3 (INPUT)
Other:
- note removed: "3.3V straigt to vbus"
